Commit message: update Engineer
A LARGE UPDATE. URDF and Controllers have been overwritten.

File: sp_description/urdf/engineer/engineer.urdf.xacro (robot description, xacro)
@@ -4,7 +4,16 @@
 	<xacro:include filename="$(find rm_description)/urdf/engineer/chassis.urdf.xacro"/>
 	<xacro:include filename="$(find sp_description)/urdf/engineer/rm_arm_transmission.xacro"/>
+	<xacro:include filename="$(find sp_description)/urdf/engineer/kinect.xacro"/>
 	<xacro:chassis roller_type="simple"/>
 	        <!--  joint  -->
 	<xacro:rm_arm/>
+	<xacro:kinect_camera prefix="camera"/>
+	<joint name="joint_camera2arm" type="fixed">
+            <axis xyz="0 0 -1"/>
+			<origin xyz="0 0 0" rpy="0 0 0"/>
+			<!--limit not work while type="continuous"-->
+            <parent link="Link_5"/>
+            <child link="camera_link"/>
+	</joint>
 	<joint name="joint_arm2body" type="fixed">
             <axis xyz="0 0 1"/>

File: sp_description/urdf/engineer/manipulator_transmission.xacro (robot description, xacro)
@@ -13,8 +13,8 @@
         </transmission>
     </xacro:macro>
-    <xacro:manipulator_transmission joint_name="Joint_1"/>
-	<xacro:manipulator_transmission joint_name="Joint_2"/>
-	<xacro:manipulator_transmission joint_name="Joint_3"/>
-	<xacro:manipulator_transmission joint_name="Joint_4"/>
-	<xacro:manipulator_transmission joint_name="Joint_5"/>
+    <xacro:manipulator_transmission joint_name="arm_joint_1"/>
+	<xacro:manipulator_transmission joint_name="arm_joint_2"/>
+	<xacro:manipulator_transmission joint_name="arm_joint_3"/>
+	<xacro:manipulator_transmission joint_name="arm_joint_4"/>
+	<xacro:manipulator_transmission joint_name="arm_joint_5"/>
 </robot>
