Commit message: manipultor类更新&整理各类文件&更新文档

File: sp_description/urdf/engineer/manipulator_transmission.xacro (robot description, xacro)
@@ -1,9 +1,9 @@
 <?xml version="1.0" encoding="utf-8"?>
 <robot xmlns:xacro="http://www.ros.org/wiki/xacro" name="engineer_manipulator">
-    <xacro:macro name="manipulator_transmission" params="joint_name">
-        <transmission name="trans_${joint_name}">
+    <xacro:macro name="manipulator_transmission" params="joint_name mechanical_reduction">
+        <transmission name="trans_${joint_name}" >
             <type>transmission_interface/SimpleTransmission</type>
             <actuator name="${joint_name}_motor">
-                <mechanicalReduction>1</mechanicalReduction>
+                <mechanicalReduction>"${mechanical_reduction}"</mechanicalReduction>
 				<hardwareInterface>hardware_interface/PositionJointInterface</hardwareInterface>
             </actuator>
@@ -13,11 +13,11 @@
         </transmission>
     </xacro:macro>
-   	<xacro:manipulator_transmission joint_name="joint1"/>
-	<xacro:manipulator_transmission joint_name="joint2"/>
-	<xacro:manipulator_transmission joint_name="joint3"/>
-	<xacro:manipulator_transmission joint_name="joint4"/>
-	<xacro:manipulator_transmission joint_name="joint5"/>
-    <xacro:manipulator_transmission joint_name="joint6"/>
-    <xacro:manipulator_transmission joint_name="joint7"/>
+   	<xacro:manipulator_transmission joint_name="joint1" mechanical_reduction="1.5"/>
+	<xacro:manipulator_transmission joint_name="joint2" mechanical_reduction="6"/>
+	<xacro:manipulator_transmission joint_name="joint3" mechanical_reduction="6"/>
+	<xacro:manipulator_transmission joint_name="joint4" mechanical_reduction="1"/>
+	<xacro:manipulator_transmission joint_name="joint5" mechanical_reduction="1"/>
+    <xacro:manipulator_transmission joint_name="joint6" mechanical_reduction="1"/>
+    <xacro:manipulator_transmission joint_name="joint7" mechanical_reduction="90.9091"/>
     <gazebo>
         <plugin name="gazebo_ros_vacuum_gripper" filename="libgazebo_ros_vacuum_gripper.so">

File: sp_description/urdf/test/rmrobot.urdf.xacro (robot description, xacro)
@@ -35,5 +35,5 @@
         </inertial>
     </link>
-    <joint name="joint1" type="prismatic">
+    <joint name="joint1" type="revolute">
         <axis xyz="0 1 0"/>
         <origin xyz="0 ${width} ${height1 - axel_offset}" rpy="0 1.57 0"/>
@@ -73,5 +73,5 @@
         <actuator name="right_front_wheel_motor">
             <hardwareInterface>hardware_interface/EffortJointInterface</hardwareInterface>
-            <mechanicalReduction>1</mechanicalReduction>
+            <mechanicalReduction>19.20</mechanicalReduction>
         </actuator>
     </transmission>
