Commit message: update URDF
Fixed a minor bug, which leads to the rviz crash. Add lidar into urdf.

File: sp_description/urdf/engineer/engineer.xacro (robot description, xacro)
@@ -5,7 +5,12 @@
 	<xacro:include filename="$(find sp_description)/urdf/engineer/fpv_module/fpv_module_test.xacro"/>
 	<xacro:include filename="$(find sp_description)/urdf/engineer/manipulator_transmission.xacro"/>
+	<xacro:include filename="$(find sp_description)/urdf/common/lidar2d.urdf.xacro"/>
+	<xacro:arg name="use_simulation" default="true"/>
 	<xacro:engineer_chassis roller_type="simple"/>
 	<xacro:engineer_manipulator/>
 	<xacro:fpv_module/>
+	<xacro:lidar2d connected_to="base_link" lidar_name="rplidar_link"
+				   simulation="$(arg use_simulation)"
+				   xyz="0.22 0 0.145" rpy="0 0 0"/>
 	<joint name="joint_arm2body" type="fixed">
 		<axis xyz="0 0 1"/>

File: sp_description/urdf/engineer/engineer_chassis/engineer_chassis.xacro (robot description, xacro)
@@ -100,6 +100,28 @@
       </geometry>
     </collision>
+  </link>
+    <xacro:mecanum_wheel prefix="left_front" connected_to="base_link"
+                         wheel_x_offset="${wheel_front}" wheel_y_offset="${wheel_left}"
+                         wheel_z_offset="${wheel_offset_z}"
+                         reflect="1" roller_type="${roller_type}"/>
+    <xacro:mecanum_wheel prefix="right_front" connected_to="base_link"
+                         wheel_x_offset="${wheel_front}" wheel_y_offset="${wheel_right}"
+                         wheel_z_offset="${wheel_offset_z}"
+                         reflect="-1" roller_type="${roller_type}"/>
+    <xacro:mecanum_wheel prefix="left_back" connected_to="base_link"
+                         wheel_x_offset="${wheel_back}" wheel_y_offset="${wheel_left}"
+                         wheel_z_offset="${wheel_offset_z}"
+                         reflect="-1" roller_type="${roller_type}"/>
+    <xacro:mecanum_wheel prefix="right_back" connected_to="base_link"
+                         wheel_x_offset="${wheel_back}" wheel_y_offset="${wheel_right}"
+                         wheel_z_offset="${wheel_offset_z}"
+                         reflect="1" roller_type="${roller_type}"/>
+    <xacro:wheel_transmission prefix="left_front" mechanical_reduction="19.2032"/>
+    <xacro:wheel_transmission prefix="right_front" mechanical_reduction="-19.2032"/>
+    <xacro:wheel_transmission prefix="left_back" mechanical_reduction="19.2032"/>
+    <xacro:wheel_transmission prefix="right_back" mechanical_reduction="-19.2032"/>
+  </xacro:macro>
 <!--swiping card link-->
-  </link>
+  <xacro:macro name="swiping_card" >
   <link
     name="swiping_card">
@@ -112,8 +134,8 @@
       <inertia
         ixx="0.00013212"
-        ixy="6.8395E-19"
-        ixz="-2.4208E-20"
+        ixy="6.8395E-06"
+        ixz="-2.4208E-06"
         iyy="0.00035298"
-        iyz="-4.3226E-11"
+        iyz="-4.3226E-06"
         izz="0.00048461" />
     </inertial>
@@ -126,9 +148,4 @@
           filename="package://sp_description/meshes/engineer_chassis/swiping_card.STL" />
       </geometry>
-      <material
-        name="">
-        <color
-          rgba="1 1 1 1" />
-      </material>
     </visual>
     <collision>
@@ -163,31 +180,10 @@
     <type>transmission_interface/SimpleTransmission</type>
     <actuator name="card_joint_motor">
-      <mechanicalReduction>1</mechanicalReduction>
-      <hardware_interface>hardware_interface/EffortJointInterface</hardware_interface>
+      <mechanicalReduction>49.97</mechanicalReduction>
     </actuator>
     <joint name="card_joint">
-      <hardware_interface>hardware_interface/EffortJointInterface</hardware_interface>
+      <hardwareInterface>hardware_interface/EffortJointInterface</hardwareInterface>
     </joint>
   </transmission>
-    <xacro:mecanum_wheel prefix="left_front" connected_to="base_link"
-                         wheel_x_offset="${wheel_front}" wheel_y_offset="${wheel_left}"
-                         wheel_z_offset="${wheel_offset_z}"
-                         reflect="1" roller_type="${roller_type}"/>
-    <xacro:mecanum_wheel prefix="right_front" connected_to="base_link"
-                         wheel_x_offset="${wheel_front}" wheel_y_offset="${wheel_right}"
-                         wheel_z_offset="${wheel_offset_z}"
-                         reflect="-1" roller_type="${roller_type}"/>
-    <xacro:mecanum_wheel prefix="left_back" connected_to="base_link"
-                         wheel_x_offset="${wheel_back}" wheel_y_offset="${wheel_left}"
-                         wheel_z_offset="${wheel_offset_z}"
-                         reflect="-1" roller_type="${roller_type}"/>
-    <xacro:mecanum_wheel prefix="right_back" connected_to="base_link"
-                         wheel_x_offset="${wheel_back}" wheel_y_offset="${wheel_right}"
-                         wheel_z_offset="${wheel_offset_z}"
-                         reflect="1" roller_type="${roller_type}"/>
-    <xacro:wheel_transmission prefix="left_front" mechanical_reduction="19.2032"/>
-    <xacro:wheel_transmission prefix="right_front" mechanical_reduction="-19.2032"/>
-    <xacro:wheel_transmission prefix="left_back" mechanical_reduction="19.2032"/>
-    <xacro:wheel_transmission prefix="right_back" mechanical_reduction="-19.2032"/>
   </xacro:macro>
 </robot>

Commit message: Add camera and fix several bugs
1. Add Vacuum, though NOT WORK.
2. Change the description.
3. Fix the bugs in fpv.

File: sp_description/urdf/engineer/engineer.xacro (robot description, xacro)
@@ -3,11 +3,12 @@
 	<xacro:include filename="$(find sp_description)/urdf/engineer/engineer_manipulator/engineer_manipulator.xacro"/>
 	<xacro:include filename="$(find sp_description)/urdf/engineer/engineer_chassis/engineer_chassis.xacro"/>
+	<xacro:include filename="$(find sp_description)/urdf/engineer/manipulator_transmission.xacro"/>
 	<xacro:include filename="$(find sp_description)/urdf/engineer/fpv_module/fpv_module_test.xacro"/>
-	<xacro:include filename="$(find sp_description)/urdf/engineer/manipulator_transmission.xacro"/>
 	<xacro:include filename="$(find sp_description)/urdf/common/lidar2d.urdf.xacro"/>
 	<xacro:arg name="use_simulation" default="true"/>
 	<xacro:engineer_chassis roller_type="simple"/>
+	<xacro:fpv_module/>
 	<xacro:engineer_manipulator/>
-	<xacro:fpv_module/>
+	<xacro:swiping_card />
 	<xacro:lidar2d connected_to="base_link" lidar_name="rplidar_front"
 				   simulation="$(arg use_simulation)"
@@ -22,11 +23,11 @@
 		<child link="arm_base_link"/>
 	</joint>
-	<joint name="joint_mast2body" type="fixed">
-		<axis xyz="0 0 1"/>
-		<origin xyz="-0.2295 -0.0815 0.0157" rpy="0 0 1.5707"/>
-		<parent link="base_link"/>
-		<child link="fpv_base_link"/>
-	</joint>
-	<gazebo>
+        <joint name="joint_mast2body" type="fixed">
+                <axis xyz="0 0 1"/>
+                <origin xyz="-0.2295 -0.0815 0.0157" rpy="0 0 1.5707"/>
+                <parent link="base_link"/>
+                <child link="fpv_base_link"/>
+        </joint>
+<gazebo>
 		<plugin name="gazebo_ros_control" filename="libgazebo_ros_control.so">
 			<robotNamespace>/</robotNamespace>

File: sp_description/urdf/engineer/engineer_manipulator/engineer_manipulator.xacro (robot description, xacro)
@@ -377,5 +377,5 @@
   <joint
     name="effector_joint"
-    type="fixed">
+    type="revolute">
     <origin
       xyz="0 0 0.0977"
@@ -386,6 +386,25 @@
       link="effector_link" />
     <axis
-      xyz="0 0 0" />
-  </joint>
- </xacro:macro>
+      xyz="0 0 1" />
+    <limit
+      lower="-1.57"
+      upper="1.57"
+      effort="2.8"
+      velocity="100" />
+  </joint>
+  <link name="grasping_frame"/>
+  <joint
+    name="grasping_frame_joint"
+    type="fixed">
+    <origin
+      xyz="0 0 0.0977"
+      rpy="0 0 0" />
+    <parent
+      link="link_5" />
+    <child
+      link="grasping_frame" />
+    <axis
+      xyz="0 0 1" />
+  </joint>
+  </xacro:macro>
 </robot>

File: sp_description/urdf/engineer/fpv_module/fpv_module.xacro (robot description, xacro)
@@ -243,5 +243,5 @@
     <type>transmission_interface/SimpleTransmission</type>
     <actuator name="fpv_pitch_joint_motor">
-      <mechanicalReduction>1</mechanicalReduction>
+	    <mechanicalReduction>1</mechanicalReduction>
     </actuator>
     <joint name="fpv_pitch_joint">
@@ -249,4 +249,43 @@
     </joint>
   </transmission>
+  <gazebo reference="fpv_pitch">
+    <material>Gazebo/Black</material>
+  </gazebo>
+        <gazebo reference="fpv_pitch">
+           <sensor type="camera" name="camera_node">
+                <update_rate>30.0</update_rate>
+                <camera name="head">
+                    <horizontal_fov>1.3962634</horizontal_fov>
+                    <image>
+                        <width>1280</width>
+                        <height>720</height>
+                        <format>R8G8B8</format>
+                    </image>
+                    <clip>
+                        <near>0.02</near>
+                        <far>300</far>
+                    </clip>
+                    <noise>
+                        <type>gaussian</type>
+                        <mean>0.0</mean>
+                        <stddev>0.007</stddev>
+                    </noise>
+                </camera>
+                <plugin name="gazebo_camera" filename="libgazebo_ros_camera.so">
+                    <alwaysOn>true</alwaysOn>
+                    <updateRate>0.0</updateRate>
+                    <cameraName>/camera</cameraName>
+                    <imageTopicName>image_raw</imageTopicName>
+                    <cameraInfoTopicName>camera_info</cameraInfoTopicName>
+                    <frameName>fpv_pitch</frameName>
+                    <hackBaseline>0.07</hackBaseline>
+                    <distortionK1>0.0</distortionK1>
+                    <distortionK2>0.0</distortionK2>
+                    <distortionK3>0.0</distortionK3>
+                    <distortionT1>0.0</distortionT1>
+                    <distortionT2>0.0</distortionT2>
+                </plugin>
+            </sensor>
+        </gazebo>
   </xacro:macro>
 </robot>

File: sp_description/urdf/engineer/fpv_module/fpv_module_test.xacro (robot description, xacro)
@@ -6,4 +6,5 @@
   name="fpv_module"
   xmlns:xacro="http://www.ros.org/wiki/xacro">
+<xacro:include filename="$(find sp_description)/urdf/engineer/fpv_module/camera.xacro"/>
   <xacro:macro name="fpv_module">
   <link
@@ -121,10 +122,10 @@
         value="0.0608808554843221" />
       <inertia
-        ixx="9.04027463419959E-06"
-        ixy="9.88988932831204E-08"
-        ixz="4.51337209267773E-08"
-        iyy="1.46381906705228E-05"
-        iyz="3.26266079201928E-07"
-        izz="1.94937658359286E-05" />
+        ixx="9.04027463419959E-03"
+        ixy="9.88988932831204E-05"
+        ixz="4.51337209267773E-05"
+        iyy="1.46381906705228E-02"
+        iyz="3.26266079201928E-04"
+        izz="1.94937658359286E-02" />
     </inertial>
     <visual>
@@ -177,8 +178,8 @@
       <inertia
         ixx="0.000904458627478079"
-        ixy="-1.04817358797102E-06"
-        ixz="3.64987845692274E-07"
+        ixy="-1.04817358797102E-03"
+        ixz="3.64987845692274E-04"
         iyy="0.00117560347818278"
-        iyz="8.43541198126057E-08"
+        iyz="8.43541198126057E-05"
         izz="0.000928104839953432" />
     </inertial>
@@ -221,4 +222,18 @@
       effort="1.3"
       velocity="6" />
+  </joint>
+  <xacro:usb_camera prefix="camera"/>
+  <joint
+    name="camera_joint"
+    type="fixed">
+    <origin
+      xyz="-0.05 -0.04 0"
+      rpy="-1.5707 0 3.1416" />
+    <parent
+      link="fpv_pitch" />
+    <child
+      link="camera_link" />
+    <axis
+      xyz="0 0 1" />
   </joint>
   <!--Transmission-->

File: sp_description/urdf/engineer/manipulator_transmission.xacro (robot description, xacro)
@@ -13,8 +13,28 @@
         </transmission>
     </xacro:macro>
-    <xacro:manipulator_transmission joint_name="arm_joint_1"/>
+   	<xacro:manipulator_transmission joint_name="arm_joint_1"/>
 	<xacro:manipulator_transmission joint_name="arm_joint_2"/>
 	<xacro:manipulator_transmission joint_name="arm_joint_3"/>
 	<xacro:manipulator_transmission joint_name="arm_joint_4"/>
 	<xacro:manipulator_transmission joint_name="arm_joint_5"/>
+    <gazebo>
+      <plugin name="gazebo_ros_vacuum_gripper" filename="libgazebo_ros_vacuum_gripper.so">
+        <robotNamespace>/effector_link</robotNamespace>
+        <bodyName>effector_link</bodyName>
+	<topicName>grasping</topicName>
+        <maxForce>100</maxForce>
+        <maxDistance>0.6</maxDistance>
+        <minDistance>0.01</minDistance>
+      </plugin>
+    </gazebo>
+    <gazebo reference="effector_link">
+        <mu1>50</mu1>
+        <mu2>50</mu2>
+ 　　　 <minDepth>0.003</minDepth>
+        <maxVel>0</maxVel>
+        <kp>10000000000000.0</kp>
+        <kd>1.0</kd>
+	<ki>2.0</ki>
+        <material>Gazebo/Grey</material>
+    </gazebo>
 </robot>

Commit message: update 20221025

File: sp_description/urdf/engineer/engineer.xacro (robot description, xacro)
@@ -13,8 +13,8 @@
 	<xacro:lidar2d connected_to="base_link" lidar_name="rplidar_front"
 				   simulation="$(arg use_simulation)"
-				   xyz="0.22 0 0.145" rpy="0 0 0"/>
+				   xyz="0.22 0 0.165" rpy="0 0 0"/>
 	<xacro:lidar2d connected_to="base_link" lidar_name="rplidar_back"
 				   simulation="$(arg use_simulation)"
-				   xyz="-0.22 0 0.145" rpy="0 0 3.14159"/>
+				   xyz="-0.22 0 0.165" rpy="0 0 3.14159"/>
 	<joint name="joint_arm2body" type="fixed">
 		<axis xyz="0 0 1"/>

File: sp_description/urdf/engineer/engineer_chassis/engineer_chassis.xacro (robot description, xacro)
@@ -53,13 +53,13 @@
     </collision>
     <collision>
-      <origin xyz="0.2375 0.0 0.13" rpy="0 0 0"/>
+      <origin xyz="0.2375 0.0 0.11" rpy="0 0 0"/>
       <geometry>
-        <box size="0.125 0.6 0.11"/>
+        <box size="0.125 0.6 0.07"/>
       </geometry>
     </collision>
     <collision>
-      <origin xyz="-0.205 0.0 0.13" rpy="0 0 0"/>
+      <origin xyz="-0.205 0.0 0.11" rpy="0 0 0"/>
       <geometry>
-        <box size="0.19 0.6 0.11"/>
+        <box size="0.19 0.6 0.07"/>
       </geometry>
     </collision>
