Commit message: 更新新工程xacro文件

File: sp_description/urdf/engineer/engineer.xacro (robot description, xacro)
@@ -4,11 +4,10 @@
 	<xacro:include filename="$(find sp_description)/urdf/engineer/engineer_chassis/engineer_chassis.xacro"/>
 	<xacro:include filename="$(find sp_description)/urdf/engineer/manipulator_transmission.xacro"/>
-	<xacro:include filename="$(find sp_description)/urdf/engineer/fpv_module/fpv_module_test.xacro"/>
-	<xacro:include filename="$(find sp_description)/urdf/common/lidar2d.urdf.xacro"/>
+	<xacro:include filename="$(find sp_description)/urdf/engineer/fpv_module/fpv_module.xacro"/>
+	<xacro:include filename="$(find sp_description)/urdf/common/lidar2d.xacro"/>
 	<xacro:arg name="use_simulation" default="true"/>
 	<xacro:engineer_chassis roller_type="simple"/>
 	<xacro:fpv_module/>
 	<xacro:engineer_manipulator/>
-	<xacro:swiping_card />
 	<xacro:lidar2d connected_to="base_link" lidar_name="rplidar_front"
 				   simulation="$(arg use_simulation)"
@@ -16,18 +15,18 @@
 	<xacro:lidar2d connected_to="base_link" lidar_name="rplidar_back"
 				   simulation="$(arg use_simulation)"
-				   xyz="-0.22 0 0.165" rpy="0 0 3.14159"/>
+				   xyz="-0.22 0 0.165" rpy="0 0 3.1416"/>
 	<joint name="joint_arm2body" type="fixed">
 		<axis xyz="0 0 1"/>
-		<origin xyz="0.0445 0.197 0.237" rpy="0 0 0"/>
+		<origin xyz="0.022 0.166 0.228" rpy="0 0 -1.5708"/>
 		<parent link="base_link"/>
 		<child link="arm_base_link"/>
 	</joint>
-        <joint name="joint_mast2body" type="fixed">
-                <axis xyz="0 0 1"/>
-                <origin xyz="-0.2295 -0.0815 0.0157" rpy="0 0 1.5707"/>
-                <parent link="base_link"/>
-                <child link="fpv_base_link"/>
-        </joint>
-<gazebo>
+	<joint name="joint_mast2body" type="fixed">
+			<axis xyz="0 0 1"/>
+			<origin xyz="-0.2295 -0.0825 0.0177" rpy="0 0 1.5708"/>
+			<parent link="base_link"/>
+			<child link="fpv_base_link"/>
+	</joint>
+	<gazebo>
 		<plugin name="gazebo_ros_control" filename="libgazebo_ros_control.so">
 			<robotNamespace>/</robotNamespace>

File: sp_description/urdf/engineer/engineer_chassis/engineer_chassis.xacro (robot description, xacro)
@@ -1,34 +1,34 @@
 <?xml version="1.0" encoding="utf-8"?>
 <!-- This URDF was automatically created by SolidWorks to URDF Exporter! Originally created by Stephen Brawner (brawner@gmail.com)
-     Commit Version: 1.5.1-0-g916b5db  Build Version: 1.5.7152.31018
+     Commit Version: 1.6.0-4-g7f85cfe  Build Version: 1.6.7995.38578
      For more information, please see http://wiki.ros.org/sw_urdf_exporter -->
 <robot
   name="engineer_chassis"
   xmlns:xacro="http://www.ros.org/wiki/xacro">
-  <xacro:include filename="$(find sp_description)/urdf/common/mecanum_wheel.urdf.xacro"/>
+  <xacro:include filename="$(find sp_description)/urdf/common/mecanum_wheel.xacro"/>
   <xacro:property name="wheel_front" value="0.19727"/>
   <xacro:property name="wheel_back" value="-0.19727"/>
-  <xacro:property name="wheel_left" value="0.223"/>
-  <xacro:property name="wheel_right" value="-0.223"/>
-  <xacro:property name="wheel_offset_z" value="-0.00111"/>
+  <xacro:property name="wheel_left" value="0.22300"/>
+  <xacro:property name="wheel_right" value="-0.22300"/>
+  <xacro:property name="wheel_offset_z" value="0.000889"/>
   <xacro:property name="wheel_joint_damping" value="1.0"/>
   <xacro:property name="wheel_joint_friction" value="1.0"/>
   <xacro:macro name="engineer_chassis" params="roller_type">
 <!--base link-->
-  <link
+   <link
     name="base_link">
     <inertial>
       <origin
-        xyz="-0.0113738412352606 -0.0179737884364999 0.0629667320671845"
+        xyz="0.0147695790883097 -0.0277071473448106 0.0578144581314767"
         rpy="0 0 0" />
       <mass
-        value="12.478309558197" />
+        value="10.0515226503987" />
       <inertia
-        ixx="0.0306729834251133"
-        ixy="2.06989089203648E-05"
-        ixz="-4.24062281514238E-06"
-        iyy="0.0340671825531538"
-        iyz="-3.89196837584769E-05"
-        izz="0.0558921594392679" />
+        ixx="0.0193511082538768"
+        ixy="-3.41760973575497E-05"
+        ixz="5.54217286706699E-06"
+        iyy="0.0356235596590244"
+        iyz="-8.92016001448171E-06"
+        izz="0.046454065978897" />
     </inertial>
     <visual>
@@ -43,5 +43,5 @@
         name="">
         <color
-          rgba="0.898039215686275 0.917647058823529 0.929411764705882 1" />
+          rgba="0.792156862745098 0.819607843137255 0.933333333333333 1" />
       </material>
     </visual>
@@ -53,49 +53,43 @@
     </collision>
     <collision>
-      <origin xyz="0.2375 0.0 0.11" rpy="0 0 0"/>
-      <geometry>
-        <box size="0.125 0.6 0.07"/>
-      </geometry>
-    </collision>
-    <collision>
-      <origin xyz="-0.205 0.0 0.11" rpy="0 0 0"/>
-      <geometry>
-        <box size="0.19 0.6 0.07"/>
-      </geometry>
-    </collision>
-    <collision>
-      <origin xyz="0.0325 0.1965 0.13" rpy="0 0 0"/>
-      <geometry>
-        <box size="0.285 0.207 0.11"/>
-      </geometry>
-    </collision>
-    <collision>
-      <origin xyz="0.0325 -0.2135 0.13" rpy="0 0 0"/>
-      <geometry>
-        <box size="0.285 0.173 0.11"/>
-      </geometry>
-    </collision>
-    <collision>
-      <origin xyz="0.0 0.2 0.21" rpy="0 0 0"/>
-      <geometry>
-        <box size="0.23 0.12 0.05"/>
-      </geometry>
-    </collision>
-    <collision>
-      <origin xyz="0.0 -0.1895 0.235" rpy="0 0 0"/>
-      <geometry>
-        <box size="0.32 0.125 0.1"/>
-      </geometry>
-    </collision>
-    <collision>
-      <origin xyz="0.0 0.098 0.25" rpy="0 0 0"/>
-      <geometry>
-        <box size="0.19 0.01 0.13" rpy="0 0 0"/>
-      </geometry>
-    </collision>
-    <collision>
-      <origin xyz="0.0 -0.132 0.3" rpy="0 0 0"/>
-      <geometry>
-        <box size="0.19 0.01 0.03"/>
+      <origin xyz="0.228 0.0 0.118" rpy="0 0 0"/>
+      <geometry>
+        <box size="0.144 0.3 0.14"/>
+      </geometry>
+    </collision>
+    <collision>
+      <origin xyz="-0.205 0.0 0.10" rpy="0 0 0"/>
+      <geometry>
+        <box size="0.19 0.3 0.09"/>
+      </geometry>
+    </collision>
+    <collision>
+      <origin xyz="-0.01 0.193 0.13" rpy="0 0 0"/>
+      <geometry>
+        <box size="0.220 0.214 0.148"/>
+      </geometry>
+    </collision>
+    <collision>
+      <origin xyz="0.0 0.22 0.09" rpy="0 0 0"/>
+      <geometry>
+        <box size="0.6 0.16 0.07"/>
+      </geometry>
+    </collision>
+    <collision>
+      <origin xyz="0.0 -0.24 0.13" rpy="0 0 0"/>
+      <geometry>
+        <box size="0.5 0.12 0.28"/>
+      </geometry>
+    </collision>
+    <collision>
+      <origin xyz="0.0 0.054 0.23" rpy="0 0 0"/>
+      <geometry>
+        <box size="0.19 0.008 0.12" rpy="0 0 0"/>
+      </geometry>
+    </collision>
+    <collision>
+      <origin xyz="0.0 -0.172 0.23" rpy="0 0 0"/>
+      <geometry>
+        <box size="0.19 0.01 0.12"/>
       </geometry>
     </collision>
@@ -122,68 +116,122 @@
     <xacro:wheel_transmission prefix="right_back" mechanical_reduction="-19.2032"/>
   </xacro:macro>
-<!--swiping card link-->
-  <xacro:macro name="swiping_card" >
-  <link
-    name="swiping_card">
-    <inertial>
-      <origin
-        xyz="-0.043679 3.1364E-15 0.0024775"
-        rpy="0 0 0" />
-      <mass
-        value="0.12034" />
-      <inertia
-        ixx="0.00013212"
-        ixy="6.8395E-06"
-        ixz="-2.4208E-06"
-        iyy="0.00035298"
-        iyz="-4.3226E-06"
-        izz="0.00048461" />
-    </inertial>
-    <visual>
-      <origin
-        xyz="0 0 0"
-        rpy="0 0 0" />
-      <geometry>
-        <mesh
-          filename="package://sp_description/meshes/engineer_chassis/swiping_card.STL" />
-      </geometry>
-    </visual>
-    <collision>
-      <origin
-        xyz="0 0 0"
-        rpy="0 0 0" />
-      <geometry>
-        <mesh
-          filename="package://sp_description/meshes/engineer_chassis/swiping_card.STL" />
-      </geometry>
-    </collision>
-  </link>
-  <joint
-    name="card_joint"
-    type="prismatic">
-    <origin
-      xyz="0.235 0 -0.0155"
-      rpy="0 0 0" />
-    <parent
-      link="base_link" />
-    <child
-      link="swiping_card" />
-    <axis
-      xyz="1 0 0" />
-    <limit
-      lower="0"
-      upper="0.2"
-      effort="80"
-      velocity="2" />
-  </joint>
-  <transmission name="trans_card_joint">
-    <type>transmission_interface/SimpleTransmission</type>
-    <actuator name="card_joint_motor">
-      <mechanicalReduction>49.97</mechanicalReduction>
-    </actuator>
-    <joint name="card_joint">
-      <hardwareInterface>hardware_interface/EffortJointInterface</hardwareInterface>
+<!--grappler link-->
+  <xacro:macro name="grappler_link">
+    <link
+      name="right_grappler">
+      <inertial>
+        <origin
+          xyz="0.0374564878439833 0.0732785925903036 -0.297577411977033"
+          rpy="0 0 0" />
+        <mass
+          value="0.129309294396376" />
+        <inertia
+          ixx="6.06808244770477E-05"
+          ixy="-1.97645234733974E-05"
+          ixz="1.18673951219721E-14"
+          iyy="3.07267845186405E-05"
+          iyz="4.37782583454494E-14"
+          izz="7.04773538349368E-05" />
+      </inertial>
+      <visual>
+        <origin
+          xyz="0 0 0"
+          rpy="0 0 0" />
+        <geometry>
+          <mesh
+            filename="package://sp_description/meshes/engineer_chassis/right_grappler.STL" />
+        </geometry>
+        <material
+          name="">
+          <color
+            rgba="0.333333333333333 0.333333333333333 0.333333333333333 1" />
+        </material>
+      </visual>
+      <collision>
+        <origin
+          xyz="0 0 0"
+          rpy="0 0 0" />
+        <geometry>
+          <mesh
+            filename="package://sp_description/meshes/engineer_chassis/right_grappler.STL" />
+        </geometry>
+      </collision>
+    </link>
+    <joint
+      name="right_grappler_joint"
+      type="revolute">
+      <origin
+        xyz="0.267500000855127 0.160000000737873 0.0513107382535401"
+        rpy="1.57079632425699 0 -3.14159265358979" />
+      <parent
+        link="base_link" />
+      <child
+        link="right_grappler" />
+      <axis
+        xyz="0 0 -1" />
+      <limit
+        lower="-3.14"
+        upper="0"
+        effort="2"
+        velocity="20" />
     </joint>
-  </transmission>
+    <link
+      name="left_grappler">
+      <inertial>
+        <origin
+          xyz="0.0355943090184279 0.0738906876241342 0.254422588217454"
+          rpy="0 0 0" />
+        <mass
+          value="0.129309294388823" />
+        <inertia
+          ixx="6.16686076407714E-05"
+          ixy="-1.99057778006741E-05"
+          ixz="1.05904460765411E-14"
+          iyy="2.97390013550263E-05"
+          iyz="4.41092234057852E-14"
+          izz="7.04773538362682E-05" />
+      </inertial>
+      <visual>
+        <origin
+          xyz="0 0 0"
+          rpy="0 0 0" />
+        <geometry>
+          <mesh
+            filename="package://sp_description/meshes/engineer_chassis/left_grappler.STL" />
+        </geometry>
+        <material
+          name="">
+          <color
+            rgba="1 1 1 1" />
+        </material>
+      </visual>
+      <collision>
+        <origin
+          xyz="0 0 0"
+          rpy="0 0 0" />
+        <geometry>
+          <mesh
+            filename="package://sp_description/meshes/engineer_chassis/left_grappler.STL" />
+        </geometry>
+      </collision>
+    </link>
+    <joint
+      name="left_grappler_joint"
+      type="revolute">
+      <origin
+        xyz="0.267563390312071 -0.116000000130697 0.0514999996038407"
+        rpy="1.57079632425699 0 3.14159265358979" />
+      <parent
+        link="base_link" />
+      <child
+        link="left_grappler" />
+      <axis
+        xyz="0 0 -1" />
+      <limit
+        lower="-3.14"
+        upper="0"
+        effort="2"
+        velocity="20" />
+    </joint>
   </xacro:macro>
 </robot>

File: sp_description/urdf/engineer/engineer_manipulator/engineer_manipulator.xacro (robot description, xacro)
@@ -4,407 +4,451 @@
      For more information, please see http://wiki.ros.org/sw_urdf_exporter -->
 <robot xmlns:xacro="http://www.ros.org/wiki/xacro" name="engineer_manipulator">
- <xacro:macro name="engineer_manipulator">
-  <link
-    name="arm_base_link">
-    <inertial>
-      <origin
-        xyz="-0.070324 5.7391E-06 0.0040174"
-        rpy="0 0 0" />
-      <mass
-        value="0.35983" />
-      <inertia
-        ixx="0.00021085"
-        ixy="1.7146E-08"
-        ixz="3.1967E-08"
-        iyy="0.00058266"
-        iyz="-4.1748E-09"
-        izz="0.00077519" />
-    </inertial>
-    <visual>
+  <xacro:macro name="engineer_manipulator">
+    <link
+      name="arm_base_link">
+      <inertial>
+        <origin
+          xyz="0.000191990525551576 -0.0379959432267828 -0.0188711762736671"
+          rpy="0 0 0" />
+        <mass
+          value="0.395354400864979" />
+        <inertia
+          ixx="0.000467726564216232"
+          ixy="-8.67714690501313E-09"
+          ixz="4.31198411045603E-09"
+          iyy="0.000307127917627802"
+          iyz="-2.40360210665882E-08"
+          izz="0.000768655424904835" />
+      </inertial>
+      <visual>
+        <origin
+          xyz="0 0 0"
+          rpy="0 0 0" />
+        <geometry>
+          <mesh
+            filename="package://sp_description/meshes/engineer_manipulator/arm_base_link.STL" />
+        </geometry>
+        <material
+          name="">
+          <color
+            rgba="0.333333333333333 0.333333333333333 0.333333333333333 1" />
+        </material>
+      </visual>
+      <collision>
+        <origin
+          xyz="0 0 0"
+          rpy="0 0 0" />
+        <geometry>
+          <mesh
+            filename="package://sp_description/meshes/engineer_manipulator/arm_base_link.STL" />
+        </geometry>
+      </collision>
+    </link>
+    <link
+      name="link1">
+      <inertial>
+        <origin
+          xyz="-0.00519778790831543 -0.000376162564114741 0.051547696306667"
+          rpy="0 0 0" />
+        <mass
+          value="0.376683384729688" />
+        <inertia
+          ixx="0.000845918540984844"
+          ixy="1.12279959742112E-07"
+          ixz="9.01688301312492E-07"
+          iyy="0.000489021055809623"
+          iyz="7.41749753688042E-07"
+          izz="0.000437357298424943" />
+      </inertial>
+      <visual>
+        <origin
+          xyz="0 0 0"
+          rpy="0 0 0" />
+        <geometry>
+          <mesh
+            filename="package://sp_description/meshes/engineer_manipulator/link1.STL" />
+        </geometry>
+        <material
+          name="">
+          <color
+            rgba="0.333333333333333 0.333333333333333 0.333333333333333 1" />
+        </material>
+      </visual>
+      <collision>
+        <origin
+          xyz="0 0 0"
+          rpy="0 0 0" />
+        <geometry>
+          <mesh
+            filename="package://sp_description/meshes/engineer_manipulator/link1.STL" />
+        </geometry>
+      </collision>
+    </link>
+    <joint
+      name="joint1"
+      type="revolute">
       <origin
         xyz="0 0 0"
         rpy="0 0 0" />
-      <geometry>
-        <mesh
-			filename="package://sp_description/meshes/engineer_manipulator/base_link.STL" />
-      </geometry>
-      <material
-        name="">
-        <color
-          rgba="0.33333 0.33333 0.33333 1" />
-      </material>
-    </visual>
-    <collision>
-      <origin
-        xyz="0 0 0"
+      <parent
+        link="arm_base_link" />
+      <child
+        link="link1" />
+      <axis
+        xyz="0 0 1" />
+      <limit
+        lower="-3.14"
+        upper="3.14"
+        effort="0"
+        velocity="0" />
+    </joint>
+    <link
+      name="link2">
+      <inertial>
+        <origin
+          xyz="0.050580281880749 1.15493250689451E-05 -0.0210030003469162"
+          rpy="0 0 0" />
+        <mass
+          value="0.759246586931641" />
+        <inertia
+          ixx="0.000476310073091113"
+          ixy="7.29764960891789E-07"
+          ixz="1.10638206714342E-07"
+          iyy="0.000991153032504733"
+          iyz="1.21515857857987E-06"
+          izz="0.00140495471373823" />
+      </inertial>
+      <visual>
+        <origin
+          xyz="0 0 0"
+          rpy="0 0 0" />
+        <geometry>
+          <mesh
+            filename="package://sp_description/meshes/engineer_manipulator/link2.STL" />
+        </geometry>
+        <material
+          name="">
+          <color
+            rgba="0.333333333333333 0.333333333333333 0.333333333333333 1" />
+        </material>
+      </visual>
+      <collision>
+        <origin
+          xyz="0 0 0"
+          rpy="0 0 0" />
+        <geometry>
+          <mesh
+            filename="package://sp_description/meshes/engineer_manipulator/link2.STL" />
+        </geometry>
+      </collision>
+    </link>
+    <joint
+      name="joint2"
+      type="revolute">
+      <origin
+        xyz="-0.022 0 0.065"
+        rpy="0 -1.5708 0" />
+      <parent
+        link="link1" />
+      <child
+        link="link2" />
+      <axis
+        xyz="0 0 -1" />
+      <limit
+        lower="-1.57"
+        upper="1.57"
+        effort="0"
+        velocity="0" />
+    </joint>
+    <link
+      name="link3">
+      <inertial>
+        <origin
+          xyz="0.0245084498465696 0.00738609929531111 0.00192882422441409"
+          rpy="0 0 0" />
+        <mass
+          value="0.728531979995667" />
+        <inertia
+          ixx="0.000532458424182733"
+          ixy="4.53824196718106E-06"
+          ixz="2.04205314034E-06"
+          iyy="0.000532510298817301"
+          iyz="-1.81917766175563E-06"
+          izz="0.000337461792942105" />
+      </inertial>
+      <visual>
+        <origin
+          xyz="0 0 0"
+          rpy="0 0 0" />
+        <geometry>
+          <mesh
+            filename="package://sp_description/meshes/engineer_manipulator/link3.STL" />
+        </geometry>
+        <material
+          name="">
+          <color
+            rgba="0.333333333333333 0.333333333333333 0.333333333333333 1" />
+        </material>
+      </visual>
+      <collision>
+        <origin
+          xyz="0 0 0"
+          rpy="0 0 0" />
+        <geometry>
+          <mesh
+            filename="package://sp_description/meshes/engineer_manipulator/link3.STL" />
+        </geometry>
+      </collision>
+    </link>
+    <joint
+      name="joint3"
+      type="revolute">
+      <origin
+        xyz="0.2 0 0"
         rpy="0 0 0" />
-      <geometry>
-        <mesh
-			filename="package://sp_description/meshes/engineer_manipulator/base_link.STL" />
-      </geometry>
-    </collision>
-  </link>
-  <link
-    name="link_1">
-    <inertial>
-      <origin
-        xyz="-7.3534E-05 0.010781 0.08501"
+      <parent
+        link="link2" />
+      <child
+        link="link3" />
+      <axis
+        xyz="0 0 1" />
+      <limit
+        lower="-1.57"
+        upper="1.57"
+        effort="0"
+        velocity="0" />
+    </joint>
+    <link
+      name="link4">
+      <inertial>
+        <origin
+          xyz="-4.15720177258799E-05 0.00320298874916644 0.00671219827123581"
+          rpy="0 0 0" />
+        <mass
+          value="0.227354423602744" />
+        <inertia
+          ixx="0.00017836251229402"
+          ixy="-4.3119850715308E-09"
+          ixz="5.53767841869846E-10"
+          iyy="0.000191169545672061"
+          iyz="2.40360190145244E-08"
+          izz="0.000327594643478463" />
+      </inertial>
+      <visual>
+        <origin
+          xyz="0 0 0"
+          rpy="0 0 0" />
+        <geometry>
+          <mesh
+            filename="package://sp_description/meshes/engineer_manipulator/link4.STL" />
+        </geometry>
+        <material
+          name="">
+          <color
+            rgba="0.823529411764706 0.870588235294118 0.980392156862745 1" />
+        </material>
+      </visual>
+      <collision>
+        <origin
+          xyz="0 0 0"
+          rpy="0 0 0" />
+        <geometry>
+          <mesh
+            filename="package://sp_description/meshes/engineer_manipulator/link4.STL" />
+        </geometry>
+      </collision>
+    </link>
+    <joint
+      name="joint4"
+      type="revolute">
+      <origin
+        xyz="0.13435 0 0"
+        rpy="0 1.5708 0" />
+      <parent
+        link="link3" />
+      <child
+        link="link4" />
+      <axis
+        xyz="0 0 1" />
+      <limit
+        lower="-3.14"
+        upper="3.14"
+        effort="0"
+        velocity="0" />
+    </joint>
+    <link
+      name="link5">
+      <inertial>
+        <origin
+          xyz="0.0448570389290742 7.50749423052491E-05 -0.0145612470233759"
+          rpy="0 0 0" />
+        <mass
+          value="0.0807348568456161" />
+        <inertia
+          ixx="3.32465515141751E-05"
+          ixy="-2.40360210662102E-08"
+          ixz="-4.31198411042277E-09"
+          iyy="2.26337327690657E-05"
+          iyz="5.39577655542099E-10"
+          izz="2.31477934401328E-05" />
+      </inertial>
+      <visual>
+        <origin
+          xyz="0 0 0"
+          rpy="0 0 0" />
+        <geometry>
+          <mesh
+            filename="package://sp_description/meshes/engineer_manipulator/link5.STL" />
+        </geometry>
+        <material
+          name="">
+          <color
+            rgba="0.792156862745098 0.819607843137255 0.933333333333333 1" />
+        </material>
+      </visual>
+      <collision>
+        <origin
+          xyz="0 0 0"
+          rpy="0 0 0" />
+        <geometry>
+          <mesh
+            filename="package://sp_description/meshes/engineer_manipulator/link5.STL" />
+        </geometry>
+      </collision>
+    </link>
+    <joint
+      name="joint5"
+      type="revolute">
+      <origin
+        xyz="0 -0.025 0.05"
+        rpy="1.5708 -1.5708 0" />
+      <parent
+        link="link4" />
+      <child
+        link="link5" />
+      <axis
+        xyz="0 0 -1" />
+      <limit
+        lower="-1.57"
+        upper="1.57"
+        effort="0"
+        velocity="0" />
+    </joint>
+    <link
+      name="link6">
+      <inertial>
+        <origin
+          xyz="-0.000654571367492234 -0.0126737517821381 -0.0332087502205121"
+          rpy="0 0 0" />
+        <mass
+          value="0.315054913435457" />
+        <inertia
+          ixx="0.000458132434965079"
+          ixy="-2.89433972150163E-10"
+          ixz="-7.33704234288827E-07"
+          iyy="0.000465485967391261"
+          iyz="-7.04854531919477E-08"
+          izz="4.75075209095847E-05" />
+      </inertial>
+      <visual>
+        <origin
+          xyz="0 0 0"
+          rpy="0 0 0" />
+        <geometry>
+          <mesh
+            filename="package://sp_description/meshes/engineer_manipulator/link6.STL" />
+        </geometry>
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