Commit message: 更新新工程xacro文件

File: sp_description/urdf/engineer/fpv_module/fpv_module.xacro (robot description, xacro)
@@ -11,40 +11,37 @@
     <inertial>
       <origin
-        xyz="-0.11049 -0.12139 0.39986"
-        rpy="0 0 0" />
-      <mass
-        value="0.31829" />
-      <inertia
-        ixx="0.00097362"
-        ixy="-1.6968E-08"
-        ixz="9.9313E-08"
-        iyy="3.9154E-05"
-        iyz="-2.2956E-07"
-        izz="0.00098287" />
-    </inertial>
-    <visual>
-      <origin
-        xyz="0 0 0"
-        rpy="0 0 0" />
-      <geometry>
-        <mesh
-          filename="package://sp_description/meshes/fpv_module/base_link.STL" />
-      </geometry>
-      <material
-        name="">
-        <color
-          rgba="0.89804 0.91765 0.92941 1" />
-      </material>
-    </visual>
-    <collision>
-      <origin xyz="-0.029 0.0 00.1213" rpy="0 0 0" />
-      <geometry>
-        <box size="0.025 0.025 0.27"/>
-      </geometry>
-    </collision>
-    <collision>
-      <origin xyz="0.0085 0.01 0.2963" rpy="0 0 0"/>
-      <geometry>
-        <box size="0.1 0.09 0.08"/>
+        xyz="-0.00792936871652137 0.000141142989662449 0.260766462339412"
+        rpy="0 0 0" />
+      <mass
+        value="0.317542464634811" />
+      <inertia
+        ixx="0.000965471374037066"
+        ixy="9.93131375188562E-08"
+        ixz="-4.59210283751836E-07"
+        iyy="0.000974644385413349"
+        iyz="-2.29555782023746E-07"
+        izz="3.90092448204564E-05" />
+    </inertial>
+    <visual>
+      <origin
+        xyz="0 0 0"
+        rpy="0 0 0" />
+      <geometry>
+        <mesh
+          filename="package://sp_description/meshes/fpv_module/fpv_base_link.STL" />
+      </geometry>
+      <material
+        name="">
+        <color
+          rgba="0.898039215686275 0.917647058823529 0.929411764705882 1" />
+      </material>
+    </visual>
+    <collision>
+      <origin
+        xyz="0 0 0"
+        rpy="0 0 0" />
+      <geometry>
+        <mesh
+          filename="package://sp_description/meshes/fpv_module/fpv_base_link.STL" />
       </geometry>
     </collision>
@@ -54,15 +51,15 @@
     <inertial>
       <origin
-        xyz="0.0071654 -0.0026446 0.22366"
-        rpy="0 0 0" />
-      <mass
-        value="0.43497" />
-      <inertia
-        ixx="0.0035278"
-        ixy="-3.1775E-06"
-        ixz="-8.4026E-08"
-        iyy="0.0036181"
-        iyz="-5.812E-09"
-        izz="0.00025229" />
+        xyz="-0.0584010828086417 -0.00159000441041939 0.273527091290577"
+        rpy="0 0 0" />
+      <mass
+        value="0.596769834435929" />
+      <inertia
+        ixx="0.00358416489838144"
+        ixy="8.93424511469642E-06"
+        ixz="-8.40259560018718E-08"
+        iyy="0.00396184957629145"
+        iyz="-5.81196895554224E-09"
+        izz="0.00062348701535612" />
     </inertial>
     <visual>
@@ -77,17 +74,14 @@
         name="">
         <color
-          rgba="0.82353 0.87059 0.98039 1" />
-      </material>
-    </visual>
-    <collision>
-      <origin xyz="0.003 0 0.1738" rpy="0 0 0" />
-      <geometry>
-        <box size="0.031 0.036 0.375"/>
-      </geometry>
-    </collision>
-    <collision>
-      <origin xyz="0.038 -0.008 0.3813" rpy="0 0 0"/>
-      <geometry>
-        <box size="0.2 0.12 0.06"/>
+          rgba="0.823529411764706 0.870588235294118 0.980392156862745 1" />
+      </material>
+    </visual>
+    <collision>
+      <origin
+        xyz="0 0 0"
+        rpy="0 0 0" />
+      <geometry>
+        <mesh
+          filename="package://sp_description/meshes/fpv_module/mast.STL" />
       </geometry>
     </collision>
@@ -97,6 +91,6 @@
     type="prismatic">
     <origin
-      xyz="-0.11887 -0.4 0.13926"
-      rpy="3.1416 0 -3.1416" />
+      xyz="0 0 0"
+      rpy="0 0 0" />
     <parent
       link="fpv_base_link" />
@@ -104,5 +98,5 @@
       link="mast" />
     <axis
-      xyz="0 0 -1" />
+      xyz="0 0 1" />
     <limit
       lower="0"
@@ -115,15 +109,15 @@
     <inertial>
       <origin
-        xyz="-0.0091696 0.044106 0.018308"
-        rpy="0 0 0" />
-      <mass
-        value="0.060881" />
-      <inertia
-        ixx="9.0403E-06"
-        ixy="9.8899E-08"
-        ixz="4.5134E-08"
-        iyy="1.4638E-05"
-        iyz="3.2627E-07"
-        izz="1.9494E-05" />
+        xyz="-0.0092103 0.044084 0.018323"
+        rpy="0 0 0" />
+      <mass
+        value="0.060612" />
+      <inertia
+        ixx="9.0201E-03"
+        ixy="1.0141E-04"
+        ixz="5.7277E-05"
+        iyy="1.4587E-02"
+        iyz="3.2725E-04"
+        izz="1.9433E-02" />
     </inertial>
     <visual>
@@ -142,7 +136,10 @@
     </visual>
     <collision>
-      <origin xyz="-0.012 -0.0055 0.4138" rpy="0 0 0" />
-      <geometry>
-        <box size="0.07 0.075 0.025"/>
+      <origin
+        xyz="0 0 0"
+        rpy="0 0 0" />
+      <geometry>
+        <mesh
+          filename="package://sp_description/meshes/fpv_module/fpv_yaw.STL" />
       </geometry>
     </collision>
@@ -159,5 +156,5 @@
       link="fpv_yaw" />
     <axis
-      xyz="0 0 -1" />
+      xyz="0 0 1" />
     <limit
       lower="-1.5708"
@@ -170,5 +167,5 @@
     <inertial>
       <origin
-        xyz="-0.017448 -0.055509 -4.0542E-05"
+        xyz="-0.017448 -0.055509 -4.0539E-05"
         rpy="0 0 0" />
       <mass
@@ -176,8 +173,8 @@
       <inertia
         ixx="0.00090446"
-        ixy="-1.0482E-06"
-        ixz="3.6499E-07"
+        ixy="-1.0482E-03"
+        ixz="3.6509E-04"
         iyy="0.0011756"
-        iyz="8.4354E-08"
+        iyz="8.4354E-05"
         izz="0.0009281" />
     </inertial>
@@ -193,11 +190,14 @@
         name="">
         <color
-          rgba="0.49804 0.49804 0.49804 1" />
-      </material>
-    </visual>
-    <collision>
-      <origin xyz="-0.007 -0.028 0.4513" rpy="0 0 0" />
-      <geometry>
-        <box size="0.11 0.07 0.05"/>
+          rgba="1 1 1 1" />
+      </material>
+    </visual>
+    <collision>
+      <origin
+        xyz="0 0 0"
+        rpy="0 0 0" />
+      <geometry>
+        <mesh
+          filename="package://sp_description/meshes/fpv_module/fpv_pitch.STL" />
       </geometry>
     </collision>
@@ -207,6 +207,6 @@
     type="revolute">
     <origin
-      xyz="0 0.0007 0.0275"
-      rpy="-1.5708 0 -3.1416" />
+      xyz="0 0.000700000000000704 0.0275"
+      rpy="-1.5707963267949 0 3.14159265358979" />
     <parent
       link="fpv_yaw" />
@@ -252,40 +252,4 @@
     <material>Gazebo/Black</material>
   </gazebo>
-        <gazebo reference="fpv_pitch">
-           <sensor type="camera" name="camera_node">
-                <update_rate>30.0</update_rate>
-                <camera name="head">
-                    <horizontal_fov>1.3962634</horizontal_fov>
-                    <image>
-                        <width>1280</width>
-                        <height>720</height>
-                        <format>R8G8B8</format>
-                    </image>
-                    <clip>
-                        <near>0.02</near>
-                        <far>300</far>
-                    </clip>
-                    <noise>
-                        <type>gaussian</type>
-                        <mean>0.0</mean>
-                        <stddev>0.007</stddev>
-                    </noise>
-                </camera>
-                <plugin name="gazebo_camera" filename="libgazebo_ros_camera.so">
-                    <alwaysOn>true</alwaysOn>
-                    <updateRate>0.0</updateRate>
-                    <cameraName>/camera</cameraName>
-                    <imageTopicName>image_raw</imageTopicName>
-                    <cameraInfoTopicName>camera_info</cameraInfoTopicName>
-                    <frameName>fpv_pitch</frameName>
-                    <hackBaseline>0.07</hackBaseline>
-                    <distortionK1>0.0</distortionK1>
-                    <distortionK2>0.0</distortionK2>
-                    <distortionK3>0.0</distortionK3>
-                    <distortionT1>0.0</distortionT1>
-                    <distortionT2>0.0</distortionT2>
-                </plugin>
-            </sensor>
-        </gazebo>
   </xacro:macro>
 </robot>

File: sp_description/urdf/engineer/manipulator_transmission.xacro (robot description, xacro)
@@ -13,28 +13,10 @@
         </transmission>
     </xacro:macro>
-   	<xacro:manipulator_transmission joint_name="arm_joint_1"/>
-	<xacro:manipulator_transmission joint_name="arm_joint_2"/>
-	<xacro:manipulator_transmission joint_name="arm_joint_3"/>
-	<xacro:manipulator_transmission joint_name="arm_joint_4"/>
-	<xacro:manipulator_transmission joint_name="arm_joint_5"/>
-    <gazebo>
-      <plugin name="gazebo_ros_vacuum_gripper" filename="libgazebo_ros_vacuum_gripper.so">
-        <robotNamespace>/effector_link</robotNamespace>
-        <bodyName>effector_link</bodyName>
-	<topicName>grasping</topicName>
-        <maxForce>100</maxForce>
-        <maxDistance>0.6</maxDistance>
-        <minDistance>0.01</minDistance>
-      </plugin>
-    </gazebo>
-    <gazebo reference="effector_link">
-        <mu1>50</mu1>
-        <mu2>50</mu2>
- 　　　 <minDepth>0.003</minDepth>
-        <maxVel>0</maxVel>
-        <kp>10000000000000.0</kp>
-        <kd>1.0</kd>
-	<ki>2.0</ki>
-        <material>Gazebo/Grey</material>
-    </gazebo>
+   	<xacro:manipulator_transmission joint_name="joint1"/>
+	<xacro:manipulator_transmission joint_name="joint2"/>
+	<xacro:manipulator_transmission joint_name="joint3"/>
+	<xacro:manipulator_transmission joint_name="joint4"/>
+	<xacro:manipulator_transmission joint_name="joint5"/>
+    <xacro:manipulator_transmission joint_name="joint6"/>
+    <xacro:manipulator_transmission joint_name="joint7"/>
 </robot>

Commit message: [Fix Bugs] MG电机无法收值 1. 并未查明原因，但似乎与hw_config电机加载顺序有关

File: sp_description/urdf/engineer/engineer.xacro (robot description, xacro)
@@ -8,5 +8,5 @@
 	<xacro:arg name="use_simulation" default="true"/>
 	<xacro:engineer_chassis roller_type="simple"/>
-	<xacro:fpv_module/>
+	<!--<xacro:fpv_module/>-->
 	<xacro:engineer_manipulator/>
 	<xacro:lidar2d connected_to="base_link" lidar_name="rplidar_front"
@@ -22,10 +22,10 @@
 		<child link="arm_base_link"/>
 	</joint>
-	<joint name="joint_mast2body" type="fixed">
+	<!--<joint name="joint_mast2body" type="fixed">
 			<axis xyz="0 0 1"/>
 			<origin xyz="-0.2295 -0.0825 0.0177" rpy="0 0 1.5708"/>
 			<parent link="base_link"/>
 			<child link="fpv_base_link"/>
-	</joint>
+	</joint>-->
 	<gazebo>
 		<plugin name="gazebo_ros_control" filename="libgazebo_ros_control.so">

File: sp_description/urdf/engineer/manipulator_transmission.xacro (robot description, xacro)
@@ -5,9 +5,9 @@
             <type>transmission_interface/SimpleTransmission</type>
             <actuator name="${joint_name}_motor">
-                <mechanicalReduction>"${mechanical_reduction}"</mechanicalReduction>
-				<hardwareInterface>hardware_interface/PositionJointInterface</hardwareInterface>
+                <mechanicalReduction>${mechanical_reduction}</mechanicalReduction>
+				<hardwareInterface>hardware_interface/EffortJointInterface</hardwareInterface>
             </actuator>
 			<joint name="${joint_name}">
-				<hardwareInterface>hardware_interface/PositionJointInterface</hardwareInterface>
+				<hardwareInterface>hardware_interface/EffortJointInterface</hardwareInterface>
 			</joint>
         </transmission>
@@ -17,7 +17,8 @@
 	<xacro:manipulator_transmission joint_name="joint3" mechanical_reduction="6"/>
 	<xacro:manipulator_transmission joint_name="joint4" mechanical_reduction="1"/>
-	<xacro:manipulator_transmission joint_name="joint5" mechanical_reduction="1"/>
+	<!--<xacro:manipulator_transmission joint_name="joint5" mechanical_reduction="1"/>
     <xacro:manipulator_transmission joint_name="joint6" mechanical_reduction="1"/>
     <xacro:manipulator_transmission joint_name="joint7" mechanical_reduction="90.9091"/>
+-->
     <gazebo>
         <plugin name="gazebo_ros_vacuum_gripper" filename="libgazebo_ros_vacuum_gripper.so">

File: sp_description/urdf/test/rmrobot.urdf.xacro (robot description, xacro)
@@ -8,9 +8,9 @@
     <xacro:property name="axel_offset" value="0.05"/> <!-- Space btw top of beam and the each joint -->
     <!-- Used for fixing robot to Gazebo 'base_link' -->
-    <!--<link name="world"/>
+    <link name="world"/>
     <joint name="fixed" type="fixed">
         <parent link="world"/>
         <child link="link1"/>
-    </joint>-->
+    </joint>
     <link name="link1">
         <collision>
@@ -35,5 +35,5 @@
         </inertial>
     </link>
-    <!--<<joint name="joint1" type="revolute">
+    <joint name="joint1" type="revolute">
         <axis xyz="0 1 0"/>
         <origin xyz="0 ${width} ${height1 - axel_offset}" rpy="0 1.57 0"/>
@@ -73,5 +73,5 @@
         <actuator name="right_front_wheel_motor">
             <hardwareInterface>hardware_interface/EffortJointInterface</hardwareInterface>
-            <mechanicalReduction>1</mechanicalReduction>
+            <mechanicalReduction>6</mechanicalReduction>
         </actuator>
     </transmission>

Commit message: 更新Scene类&更新说明文档
参考说明文档，现在可以在Gazebo中飙车而不用担心创死人了

File: sp_description/urdf/engineer/engineer.xacro (robot description, xacro)
@@ -8,5 +8,5 @@
 	<xacro:arg name="use_simulation" default="true"/>
 	<xacro:engineer_chassis roller_type="simple"/>
-	<!--<xacro:fpv_module/>-->
+	<xacro:fpv_module/>
 	<xacro:engineer_manipulator/>
 	<xacro:lidar2d connected_to="base_link" lidar_name="rplidar_front"
@@ -22,10 +22,10 @@
 		<child link="arm_base_link"/>
 	</joint>
-	<!--<joint name="joint_mast2body" type="fixed">
+	<joint name="joint_mast2body" type="fixed">
 			<axis xyz="0 0 1"/>
 			<origin xyz="-0.2295 -0.0825 0.0177" rpy="0 0 1.5708"/>
 			<parent link="base_link"/>
 			<child link="fpv_base_link"/>
-	</joint>-->
+	</joint>
 	<gazebo>
 		<plugin name="gazebo_ros_control" filename="libgazebo_ros_control.so">

File: sp_description/urdf/engineer/manipulator_transmission.xacro (robot description, xacro)
@@ -6,8 +6,8 @@
             <actuator name="${joint_name}_motor">
                 <mechanicalReduction>${mechanical_reduction}</mechanicalReduction>
-				<hardwareInterface>hardware_interface/EffortJointInterface</hardwareInterface>
+				<hardwareInterface>hardware_interface/PositionJointInterface</hardwareInterface>
             </actuator>
 			<joint name="${joint_name}">
-				<hardwareInterface>hardware_interface/EffortJointInterface</hardwareInterface>
+				<hardwareInterface>hardware_interface/PositionJointInterface</hardwareInterface>
 			</joint>
         </transmission>

Commit message: update manipulator

File: sp_description/urdf/engineer/engineer.xacro (robot description, xacro)
@@ -4,16 +4,16 @@
 	<xacro:include filename="$(find sp_description)/urdf/engineer/engineer_chassis/engineer_chassis.xacro"/>
 	<xacro:include filename="$(find sp_description)/urdf/engineer/manipulator_transmission.xacro"/>
-	<xacro:include filename="$(find sp_description)/urdf/engineer/fpv_module/fpv_module.xacro"/>
-	<xacro:include filename="$(find sp_description)/urdf/common/lidar2d.xacro"/>
+	<!--<xacro:include filename="$(find sp_description)/urdf/engineer/fpv_module/fpv_module.xacro"/>
+	<xacro:include filename="$(find sp_description)/urdf/common/lidar2d.xacro"/>-->
 	<xacro:arg name="use_simulation" default="true"/>
 	<xacro:engineer_chassis roller_type="simple"/>
-	<xacro:fpv_module/>
+	<!--<xacro:fpv_module/>-->
 	<xacro:engineer_manipulator/>
-	<xacro:lidar2d connected_to="base_link" lidar_name="rplidar_front"
+	<!--<xacro:lidar2d connected_to="base_link" lidar_name="rplidar_front"
 				   simulation="$(arg use_simulation)"
 				   xyz="0.22 0 0.165" rpy="0 0 0"/>
 	<xacro:lidar2d connected_to="base_link" lidar_name="rplidar_back"
 				   simulation="$(arg use_simulation)"
-				   xyz="-0.22 0 0.165" rpy="0 0 3.1416"/>
+				   xyz="-0.22 0 0.165" rpy="0 0 3.1416"/>-->
 	<joint name="joint_arm2body" type="fixed">
 		<axis xyz="0 0 1"/>
@@ -22,10 +22,10 @@
 		<child link="arm_base_link"/>
 	</joint>
-	<joint name="joint_mast2body" type="fixed">
+	<!--<joint name="joint_mast2body" type="fixed">
 			<axis xyz="0 0 1"/>
 			<origin xyz="-0.2295 -0.0825 0.0177" rpy="0 0 1.5708"/>
 			<parent link="base_link"/>
 			<child link="fpv_base_link"/>
-	</joint>
+	</joint>-->
 	<gazebo>
 		<plugin name="gazebo_ros_control" filename="libgazebo_ros_control.so">

File: sp_description/urdf/engineer/engineer_manipulator/engineer_manipulator.xacro (robot description, xacro)
@@ -330,6 +330,6 @@
         xyz="0 0 1" />
       <limit
-        lower="-1.90"
-        upper="1.90"
+        lower="-2.10"
+        upper="2.10"
         effort="20"
         velocity="5" />

File: sp_description/urdf/engineer/manipulator_transmission.xacro (robot description, xacro)
@@ -6,8 +6,8 @@
             <actuator name="${joint_name}_motor">
                 <mechanicalReduction>${mechanical_reduction}</mechanicalReduction>
-				<hardwareInterface>hardware_interface/PositionJointInterface</hardwareInterface>
+				<hardwareInterface>hardware_interface/EffortJointInterface</hardwareInterface>
             </actuator>
 			<joint name="${joint_name}">
-				<hardwareInterface>hardware_interface/PositionJointInterface</hardwareInterface>
+				<hardwareInterface>hardware_interface/EffortJointInterface</hardwareInterface>
 			</joint>
         </transmission>
@@ -19,5 +19,5 @@
 	<xacro:manipulator_transmission joint_name="joint5" mechanical_reduction="1"/>
     <xacro:manipulator_transmission joint_name="joint6" mechanical_reduction="1"/>
-    <xacro:manipulator_transmission joint_name="joint7" mechanical_reduction="90.9091"/>
+    <xacro:manipulator_transmission joint_name="joint7" mechanical_reduction="1570.80"/>
     <gazebo>
         <plugin name="gazebo_ros_vacuum_gripper" filename="libgazebo_ros_vacuum_gripper.so">

File: sp_description/urdf/test/rmrobot.urdf.xacro (robot description, xacro)
@@ -35,5 +35,5 @@
         </inertial>
     </link>
-    <joint name="joint1" type="revolute">
+    <joint name="joint1" type="prismatic">
         <axis xyz="0 1 0"/>
         <origin xyz="0 ${width} ${height1 - axel_offset}" rpy="0 1.57 0"/>
@@ -65,5 +65,5 @@
                     izz="${mass / 12.0 * (width*width + width*width)}"/>
         </inertial>
-    </link>-->
+    </link>
     <transmission name="tran1">
         <type>transmission_interface/SimpleTransmission</type>
@@ -73,5 +73,5 @@
         <actuator name="right_front_wheel_motor">
             <hardwareInterface>hardware_interface/EffortJointInterface</hardwareInterface>
-            <mechanicalReduction>6</mechanicalReduction>
+            <mechanicalReduction>1570.80</mechanicalReduction>
         </actuator>
     </transmission>

Commit message: Update some remote controling

File: sp_description/urdf/engineer/engineer.xacro (robot description, xacro)
@@ -4,16 +4,9 @@
 	<xacro:include filename="$(find sp_description)/urdf/engineer/engineer_chassis/engineer_chassis.xacro"/>
 	<xacro:include filename="$(find sp_description)/urdf/engineer/manipulator_transmission.xacro"/>
-	<!--<xacro:include filename="$(find sp_description)/urdf/engineer/fpv_module/fpv_module.xacro"/>
-	<xacro:include filename="$(find sp_description)/urdf/common/lidar2d.xacro"/>-->
+	<xacro:include filename="$(find sp_description)/urdf/engineer/fpv_module/fpv_module.xacro"/>
 	<xacro:arg name="use_simulation" default="true"/>
 	<xacro:engineer_chassis roller_type="simple"/>
-	<!--<xacro:fpv_module/>-->
+	<xacro:fpv_module/>
 	<xacro:engineer_manipulator/>
-	<!--<xacro:lidar2d connected_to="base_link" lidar_name="rplidar_front"
-				   simulation="$(arg use_simulation)"
-				   xyz="0.22 0 0.165" rpy="0 0 0"/>
-	<xacro:lidar2d connected_to="base_link" lidar_name="rplidar_back"
-				   simulation="$(arg use_simulation)"
-				   xyz="-0.22 0 0.165" rpy="0 0 3.1416"/>-->
 	<joint name="joint_arm2body" type="fixed">
 		<axis xyz="0 0 1"/>
@@ -22,10 +15,10 @@
 		<child link="arm_base_link"/>
 	</joint>
-	<!--<joint name="joint_mast2body" type="fixed">
+	<joint name="joint_mast2body" type="fixed">
 			<axis xyz="0 0 1"/>
 			<origin xyz="-0.2295 -0.0825 0.0177" rpy="0 0 1.5708"/>
 			<parent link="base_link"/>
 			<child link="fpv_base_link"/>
-	</joint>-->
+	</joint>
 	<gazebo>
 		<plugin name="gazebo_ros_control" filename="libgazebo_ros_control.so">

File: sp_description/urdf/engineer/fpv_module/fpv_module.xacro (robot description, xacro)
@@ -150,5 +150,5 @@
     <origin
       xyz="0 -0.0285 0.3853"
-      rpy="0 0 0" />
+      rpy="0 0 -1.5707963267949" />
     <parent
       link="mast" />

File: sp_description/urdf/engineer/manipulator_transmission.xacro (robot description, xacro)
@@ -6,8 +6,8 @@
             <actuator name="${joint_name}_motor">
                 <mechanicalReduction>${mechanical_reduction}</mechanicalReduction>
-				<hardwareInterface>hardware_interface/EffortJointInterface</hardwareInterface>
+				<hardwareInterface>hardware_interface/PositionJointInterface</hardwareInterface>
             </actuator>
 			<joint name="${joint_name}">
-				<hardwareInterface>hardware_interface/EffortJointInterface</hardwareInterface>
+				<hardwareInterface>hardware_interface/PositionJointInterface</hardwareInterface>
 			</joint>
         </transmission>
