Commit message: pid

File: sp_description/urdf/engineer/engineer.xacro (robot description, xacro)
@@ -3,12 +3,11 @@
 	<xacro:include filename="$(find sp_description)/urdf/engineer/engineer_manipulator/engineer_manipulator.xacro"/>
 	<xacro:include filename="$(find sp_description)/urdf/engineer/engineer_chassis/engineer_chassis.xacro"/>
-	<!--<xacro:include filename="$(find sp_description)/urdf/engineer/manipulator_transmission.xacro"/>
-	<xacro:include filename="$(find sp_description)/urdf/engineer/fpv_module/fpv_module.xacro"/>
+	<xacro:include filename="$(find sp_description)/urdf/engineer/manipulator_transmission.xacro"/>
+	<!--<xacro:include filename="$(find sp_description)/urdf/engineer/fpv_module/fpv_module.xacro"/>
 -->
 	<xacro:arg name="use_simulation" default="true"/>
 	<xacro:engineer_chassis roller_type="simple"/>
-	<!--<xacro:fpv_module/>
-	<xacro:engineer_manipulator/>-->
-<!--
+	<!--<xacro:fpv_module/>-->
+	<xacro:engineer_manipulator/>
 	<joint name="joint_arm2body" type="fixed">
 		<axis xyz="0 0 1"/>
@@ -17,5 +16,5 @@
 		<child link="arm_base_link"/>
 	</joint>
-	<joint name="joint_mast2body" type="fixed">
+	<!--<joint name="joint_mast2body" type="fixed">
 			<axis xyz="0 0 1"/>
 			<origin xyz="-0.2295 -0.0825 0.0177" rpy="0 0 1.5708"/>

File: sp_description/urdf/engineer/engineer_chassis/engineer_chassis.xacro (robot description, xacro)
@@ -111,8 +111,8 @@
                          wheel_z_offset="${wheel_offset_z}"
                          reflect="1" roller_type="${roller_type}"/>
-    <xacro:wheel_transmission prefix="left_front" mechanical_reduction="19.2032"/>
+    <!--<xacro:wheel_transmission prefix="left_front" mechanical_reduction="19.2032"/>
     <xacro:wheel_transmission prefix="right_front" mechanical_reduction="-19.2032"/>
     <xacro:wheel_transmission prefix="left_back" mechanical_reduction="19.2032"/>
-    <xacro:wheel_transmission prefix="right_back" mechanical_reduction="-19.2032"/>
+    <xacro:wheel_transmission prefix="right_back" mechanical_reduction="-19.2032"/>-->
   </xacro:macro>
 <!--grappler link-->

File: sp_description/urdf/engineer/engineer_manipulator/engineer_manipulator.xacro (robot description, xacro)
@@ -388,6 +388,6 @@
       xyz="0 0 1" />
     <limit
-      lower="-1.57"
-      upper="1.57"
+      lower="-3.14"
+      upper="3.14"
       effort="20"
       velocity="5" />

Commit message: 更新键盘发送gpio&判断合适机械臂路径
待测

File: sp_description/urdf/engineer/engineer.xacro (robot description, xacro)
@@ -3,12 +3,10 @@
 	<xacro:include filename="$(find sp_description)/urdf/engineer/engineer_manipulator/engineer_manipulator.xacro"/>
 	<xacro:include filename="$(find sp_description)/urdf/engineer/engineer_chassis/engineer_chassis.xacro"/>
-	<!--<xacro:include filename="$(find sp_description)/urdf/engineer/manipulator_transmission.xacro"/>
-	<xacro:include filename="$(find sp_description)/urdf/engineer/fpv_module/fpv_module.xacro"/>
--->
+	<xacro:include filename="$(find sp_description)/urdf/engineer/manipulator_transmission.xacro"/>
+	<!--xacro:include filename="$(find sp_description)/urdf/engineer/fpv_module/fpv_module.xacro"/>-->
 	<xacro:arg name="use_simulation" default="true"/>
 	<xacro:engineer_chassis roller_type="simple"/>
-	<!--<xacro:fpv_module/>
-	<xacro:engineer_manipulator/>-->
-<!--
+	<!--<xacro:fpv_module/>-->
+	<xacro:engineer_manipulator/>
 	<joint name="joint_arm2body" type="fixed">
 		<axis xyz="0 0 1"/>
@@ -17,5 +15,5 @@
 		<child link="arm_base_link"/>
 	</joint>
-	<joint name="joint_mast2body" type="fixed">
+	<!--<joint name="joint_mast2body" type="fixed">
 			<axis xyz="0 0 1"/>
 			<origin xyz="-0.2295 -0.0825 0.0177" rpy="0 0 1.5708"/>

File: sp_description/urdf/engineer/engineer_chassis/engineer_chassis.xacro (robot description, xacro)
@@ -111,8 +111,8 @@
                          wheel_z_offset="${wheel_offset_z}"
                          reflect="1" roller_type="${roller_type}"/>
-    <xacro:wheel_transmission prefix="left_front" mechanical_reduction="19.2032"/>
+    <!--<xacro:wheel_transmission prefix="left_front" mechanical_reduction="19.2032"/>
     <xacro:wheel_transmission prefix="right_front" mechanical_reduction="-19.2032"/>
     <xacro:wheel_transmission prefix="left_back" mechanical_reduction="19.2032"/>
-    <xacro:wheel_transmission prefix="right_back" mechanical_reduction="-19.2032"/>
+    <xacro:wheel_transmission prefix="right_back" mechanical_reduction="-19.2032"/>-->
   </xacro:macro>
 <!--grappler link-->

File: sp_description/urdf/engineer/engineer_manipulator/engineer_manipulator.xacro (robot description, xacro)
@@ -388,6 +388,6 @@
       xyz="0 0 1" />
     <limit
-      lower="-1.57"
-      upper="1.57"
+      lower="-3.14"
+      upper="3.14"
       effort="20"
       velocity="5" />
@@ -456,5 +456,5 @@
       type="fixed">
       <origin
-        xyz="0 0 0.048"
+        xyz="0 0 0.055"
         rpy="0 0 0" />
       <parent

Commit message: Update Gpio && Gpio completed

File: sp_description/urdf/engineer/engineer.xacro (robot description, xacro)
@@ -1,24 +1,24 @@
 <?xml version="1.0"?>
 <robot xmlns:xacro="http://www.ros.org/wiki/xacro" name="engineer">
-	<xacro:include filename="$(find sp_description)/urdf/engineer/engineer_manipulator/engineer_manipulator.xacro"/>
+	<!--<xacro:include filename="$(find sp_description)/urdf/engineer/engineer_manipulator/engineer_manipulator.xacro"/>-->
 	<xacro:include filename="$(find sp_description)/urdf/engineer/engineer_chassis/engineer_chassis.xacro"/>
-	<xacro:include filename="$(find sp_description)/urdf/engineer/manipulator_transmission.xacro"/>
-	<!--xacro:include filename="$(find sp_description)/urdf/engineer/fpv_module/fpv_module.xacro"/>-->
+	<!--<xacro:include filename="$(find sp_description)/urdf/engineer/manipulator_transmission.xacro"/>-->
+	<xacro:include filename="$(find sp_description)/urdf/engineer/fpv_module/fpv_module.xacro"/>
 	<xacro:arg name="use_simulation" default="true"/>
 	<xacro:engineer_chassis roller_type="simple"/>
-	<!--<xacro:fpv_module/>-->
-	<xacro:engineer_manipulator/>
-	<joint name="joint_arm2body" type="fixed">
+	<xacro:fpv_module/>
+	<!--<xacro:engineer_manipulator/>-->
+	<!--<joint name="joint_arm2body" type="fixed">
 		<axis xyz="0 0 1"/>
 		<origin xyz="0.022 0.166 0.228" rpy="0 0 -1.5708"/>
 		<parent link="base_link"/>
 		<child link="arm_base_link"/>
-	</joint>
-	<!--<joint name="joint_mast2body" type="fixed">
+	</joint>-->
+	<joint name="joint_mast2body" type="fixed">
 			<axis xyz="0 0 1"/>
 			<origin xyz="-0.2295 -0.0825 0.0177" rpy="0 0 1.5708"/>
 			<parent link="base_link"/>
 			<child link="fpv_base_link"/>
-	</joint>-->
+	</joint>
 	<gazebo>
 		<plugin name="gazebo_ros_control" filename="libgazebo_ros_control.so">

File: sp_description/urdf/engineer/engineer_chassis/engineer_chassis.xacro (robot description, xacro)
@@ -111,8 +111,8 @@
                          wheel_z_offset="${wheel_offset_z}"
                          reflect="1" roller_type="${roller_type}"/>
-    <!--<xacro:wheel_transmission prefix="left_front" mechanical_reduction="19.2032"/>
+    <xacro:wheel_transmission prefix="left_front" mechanical_reduction="19.2032"/>
     <xacro:wheel_transmission prefix="right_front" mechanical_reduction="-19.2032"/>
     <xacro:wheel_transmission prefix="left_back" mechanical_reduction="19.2032"/>
-    <xacro:wheel_transmission prefix="right_back" mechanical_reduction="-19.2032"/>-->
+    <xacro:wheel_transmission prefix="right_back" mechanical_reduction="-19.2032"/>
   </xacro:macro>
 <!--grappler link-->

File: sp_description/urdf/test/rmrobot.xacro (robot description, xacro)
@@ -73,5 +73,5 @@
         <actuator name="right_front_wheel_motor">
             <hardwareInterface>hardware_interface/EffortJointInterface</hardwareInterface>
-            <mechanicalReduction>1</mechanicalReduction>
+            <mechanicalReduction>50</mechanicalReduction>
         </actuator>
     </transmission>

Commit message: 紧急回调l5~l7模型&修改不往1ff帧中写值的bug

File: sp_description/urdf/engineer/engineer.xacro (robot description, xacro)
@@ -1,18 +1,18 @@
 <?xml version="1.0"?>
 <robot xmlns:xacro="http://www.ros.org/wiki/xacro" name="engineer">
-	<!--<xacro:include filename="$(find sp_description)/urdf/engineer/engineer_manipulator/engineer_manipulator.xacro"/>-->
+	<xacro:include filename="$(find sp_description)/urdf/engineer/engineer_manipulator/engineer_manipulator.xacro"/>
 	<xacro:include filename="$(find sp_description)/urdf/engineer/engineer_chassis/engineer_chassis.xacro"/>
-	<!--<xacro:include filename="$(find sp_description)/urdf/engineer/manipulator_transmission.xacro"/>-->
+	<xacro:include filename="$(find sp_description)/urdf/engineer/manipulator_transmission.xacro"/>
 	<xacro:include filename="$(find sp_description)/urdf/engineer/fpv_module/fpv_module.xacro"/>
 	<xacro:arg name="use_simulation" default="true"/>
 	<xacro:engineer_chassis roller_type="simple"/>
 	<xacro:fpv_module/>
-	<!--<xacro:engineer_manipulator/>-->
-	<!--<joint name="joint_arm2body" type="fixed">
+	<xacro:engineer_manipulator/>
+	<joint name="joint_arm2body" type="fixed">
 		<axis xyz="0 0 1"/>
 		<origin xyz="0.022 0.166 0.228" rpy="0 0 -1.5708"/>
 		<parent link="base_link"/>
 		<child link="arm_base_link"/>
-	</joint>-->
+	</joint>
 	<joint name="joint_mast2body" type="fixed">
 			<axis xyz="0 0 1"/>

File: sp_description/urdf/engineer/fpv_module/fpv_module.xacro (robot description, xacro)
@@ -98,8 +98,8 @@
       link="mast" />
     <axis
-      xyz="0 0 -1" />
+      xyz="0 0 1" />
     <limit
       lower="0"
-      upper="0.235"
+      upper="0.218"
       effort="50"
       velocity="0.8" />

File: sp_description/urdf/test/rmrobot.xacro (robot description, xacro)
@@ -73,5 +73,5 @@
         <actuator name="right_front_wheel_motor">
             <hardwareInterface>hardware_interface/EffortJointInterface</hardwareInterface>
-            <mechanicalReduction>50</mechanicalReduction>
+            <mechanicalReduction>1</mechanicalReduction>
         </actuator>
     </transmission>
