Commit message: Update 20221215
1. 运动学重写。很多与样车坐标系不同的敌方并没有考虑进去，目前仿真中旋转仍不能实现。！！代码不能直接照搬的！！或者按样机坐标系调整urdf，又或者按照urdf调整坐标系,，总之请重写
2. 启动按此顺序：
    * roslaunch engineer_gazebo sentry_bringup_sim.launch
    * roslaunch chassis_controller chassis_controller_load.launch
3. PID 需要整定
4. 关于engineer_gazebo包名，后续会独立出来，并重新命名为gezebo_sim的，不用重新建立sentry_gazebo功能包
5. 考虑到后续会有gimbal，建议urdf内按sentry/swerve_chassis/*命名而非sentry/swerve_sentry_v1/*
6. 我调整了urdf内所有与joint有关的命名（保持格式整洁）

File: sp_description/urdf/sentry/swerve_sentry_v1/swerve_sentry_v1.urdf.xacro (robot description, xacro)
@@ -6,4 +6,8 @@
   name="swerve_sentry_v1"
   xmlns:xacro="http://www.ros.org/wiki/xacro">
+  <xacro:property name="driving_jnt_eff_limit" value="10"/>
+  <xacro:property name="driving_jnt_vel_limit" value="70"/>
+  <xacro:property name="heading_jnt_eff_limit" value="12"/>
+  <xacro:property name="heading_jnt_vel_limit" value="50"/>
   <link
     name="base_link">
@@ -87,5 +91,5 @@
   </link>
   <joint
-    name="swerve_back_left_joint"
+    name="left_back_heading_joint"
     type="revolute">
     <origin
@@ -98,9 +102,5 @@
     <axis
       xyz="0 0 -1" />
-    <limit
-      lower="0"
-      upper="0"
-      effort="0"
-      velocity="0" />
+    <limit lower="-1e9" upper="1e9" effort="${heading_jnt_eff_limit}" velocity="${heading_jnt_vel_limit}" />
   </joint>
   <link
@@ -145,5 +145,5 @@
   </link>
   <joint
-    name="driving_back_left_joint"
+    name="left_back_driving_joint"
     type="revolute">
     <origin
@@ -156,9 +156,5 @@
     <axis
       xyz="0 0 -1" />
-    <limit
-      lower="0"
-      upper="0"
-      effort="0"
-      velocity="0" />
+    <limit lower="-1e9" upper="1e9" effort="${driving_jnt_eff_limit}" velocity="${driving_jnt_vel_limit}" />
   </joint>
   <link
@@ -203,5 +199,5 @@
   </link>
   <joint
-    name="swerve_back_right_joint"
+    name="right_back_heading_joint"
     type="revolute">
     <origin
@@ -214,9 +210,5 @@
     <axis
       xyz="0 0 -1" />
-    <limit
-      lower="0"
-      upper="0"
-      effort="0"
-      velocity="0" />
+    <limit lower="-1e9" upper="1e9" effort="${heading_jnt_eff_limit}" velocity="${heading_jnt_vel_limit}" />
   </joint>
   <link
@@ -261,5 +253,5 @@
   </link>
   <joint
-    name="driving_back_right_joint"
+    name="right_back_driving_joint"
     type="revolute">
     <origin
@@ -272,9 +264,5 @@
     <axis
       xyz="0 0 -1" />
-    <limit
-      lower="0"
-      upper="0"
-      effort="0"
-      velocity="0" />
+    <limit lower="-1e9" upper="1e9" effort="${driving_jnt_eff_limit}" velocity="${driving_jnt_vel_limit}" />
   </joint>
   <link
@@ -319,5 +307,5 @@
   </link>
   <joint
-    name="swerve_heading_right_joint"
+    name="right_front_heading_joint"
     type="revolute">
     <origin
@@ -330,9 +318,5 @@
     <axis
       xyz="0 0 1" />
-    <limit
-      lower="0"
-      upper="0"
-      effort="0"
-      velocity="0" />
+    <limit lower="-1e9" upper="1e9" effort="${heading_jnt_eff_limit}" velocity="${heading_jnt_vel_limit}" />
   </joint>
   <link
@@ -377,5 +361,5 @@
   </link>
   <joint
-    name="driving_heading_right_joint"
+    name="right_front_driving_joint"
     type="revolute">
     <origin
@@ -388,9 +372,5 @@
     <axis
       xyz="0 0 -1" />
-    <limit
-      lower="0"
-      upper="0"
-      effort="0"
-      velocity="0" />
+    <limit lower="-1e9" upper="1e9" effort="${driving_jnt_eff_limit}" velocity="${driving_jnt_vel_limit}" />
   </joint>
   <link
@@ -435,5 +415,5 @@
   </link>
   <joint
-    name="swerve_heading_left_joint"
+    name="left_front_heading_joint"
     type="revolute">
     <origin
@@ -446,9 +426,5 @@
     <axis
       xyz="0 0 1" />
-    <limit
-      lower="0"
-      upper="0"
-      effort="0"
-      velocity="0" />
+    <limit lower="-1e9" upper="1e9" effort="${heading_jnt_eff_limit}" velocity="${heading_jnt_vel_limit}" />
   </joint>
   <link
@@ -493,5 +469,5 @@
   </link>
   <joint
-    name="driving_heading_left_joint"
+    name="left_front_driving_joint"
     type="revolute">
     <origin
@@ -504,86 +480,29 @@
     <axis
       xyz="0 0 -1" />
-    <limit
-      lower="0"
-      upper="0"
-      effort="0"
-      velocity="0" />
-  </joint>
-<!-- transmission for back_left_wheel -->
-  <transmission name="trans_swerve_back_left_joint">
-    <type>transmission_interface/SimpleTransmission</type>
-    <actuator name="swerve_back_left_actuator">
-      <mechanicalReduction>1</mechanicalReduction>
-    </actuator>
-    <joint name="swerve_back_left_joint">
-      <hardwareInterface>hardware_interface/EffortJointInterface</hardwareInterface>
-    </joint>
-  </transmission>
-  <transmission name="trans_driving_back_left_joint">
-    <type>transmission_interface/SimpleTransmission</type>
-    <actuator name="driving_back_left_actuator">
-      <mechanicalReduction>1</mechanicalReduction>
-    </actuator>
-    <joint name="driving_back_left_joint">
-      <hardwareInterface>hardware_interface/EffortJointInterface</hardwareInterface>
-    </joint>
-  </transmission>
-<!-- transmission for back_right_wheel -->
-  <transmission name="trans_swerve_back_right_joint">
-    <type>transmission_interface/SimpleTransmission</type>
-    <actuator name="swerve_back_right_actuator">
-      <mechanicalReduction>1</mechanicalReduction>
-    </actuator>
-    <joint name="swerve_back_right_joint">
-      <hardwareInterface>hardware_interface/EffortJointInterface</hardwareInterface>
-    </joint>
-  </transmission>
-  <transmission name="trans_driving_back_right_joint">
-    <type>transmission_interface/SimpleTransmission</type>
-    <actuator name="driving_back_right_actuator">
-      <mechanicalReduction>1</mechanicalReduction>
-    </actuator>
-    <joint name="driving_back_right_joint">
-      <hardwareInterface>hardware_interface/EffortJointInterface</hardwareInterface>
-    </joint>
-  </transmission>
-<!-- transmission for heading_right_wheel -->
-  <transmission name="trans_swerve_heading_right_joint">
-    <type>transmission_interface/SimpleTransmission</type>
-    <actuator name="swerve_heading_right_actuator">
-      <mechanicalReduction>1</mechanicalReduction>
-    </actuator>
-    <joint name="swerve_heading_right_joint">
-      <hardwareInterface>hardware_interface/EffortJointInterface</hardwareInterface>
-    </joint>
-  </transmission>
-  <transmission name="trans_driving_heading_right_joint">
-    <type>transmission_interface/SimpleTransmission</type>
-    <actuator name="driving_heading_right_actuator">
-      <mechanicalReduction>1</mechanicalReduction>
-    </actuator>
-    <joint name="driving_heading_right_joint">
-      <hardwareInterface>hardware_interface/EffortJointInterface</hardwareInterface>
-    </joint>
-  </transmission>
-<!-- transmission for heading_left_wheel -->
-  <transmission name="trans_swerve_heading_left_joint">
-    <type>transmission_interface/SimpleTransmission</type>
-    <actuator name="swerve_heading_left_actuator">
-      <mechanicalReduction>1</mechanicalReduction>
-    </actuator>
-    <joint name="swerve_heading_left_joint">
-      <hardwareInterface>hardware_interface/EffortJointInterface</hardwareInterface>
-    </joint>
-  </transmission>
-  <transmission name="trans_driving_heading_left_joint">
-    <type>transmission_interface/SimpleTransmission</type>
-    <actuator name="driving_heading_left_actuator">
-      <mechanicalReduction>1</mechanicalReduction>
-    </actuator>
-    <joint name="driving_heading_left_joint">
-      <hardwareInterface>hardware_interface/EffortJointInterface</hardwareInterface>
-    </joint>
-  </transmission>
+    <limit lower="-1e9" upper="1e9" effort="${driving_jnt_eff_limit}" velocity="${driving_jnt_vel_limit}" />
+  </joint>
+  <xacro:macro name="joint_transmission" params="prefix">
+    <transmission name="trans_${prefix}">
+      <type>transmission_interface/SimpleTransmission</type>
+      <actuator name="${prefix}_actuator">
+        <mechanicalReduction>1</mechanicalReduction>
+      </actuator>
+      <joint name="${prefix}_joint">
+        <hardwareInterface>hardware_interface/EffortJointInterface</hardwareInterface>
+      </joint>
+    </transmission>
+  </xacro:macro>
+<!-- transmission for left_back_wheel-->
+  <xacro:joint_transmission prefix="left_back_heading"/>
+  <xacro:joint_transmission prefix="left_back_driving"/>
+<!-- transmission for right_back_wheel-->
+  <xacro:joint_transmission prefix="right_back_heading"/>
+  <xacro:joint_transmission prefix="right_back_driving"/>
+<!-- transmission for right_front_wheel-->
+  <xacro:joint_transmission prefix="right_front_heading"/>
+  <xacro:joint_transmission prefix="right_front_driving"/>
+<!-- transmission for left_front_wheel -->
+  <xacro:joint_transmission prefix="left_front_heading"/>
+  <xacro:joint_transmission prefix="left_front_driving"/>
 <!-- gazebo config -->
   <gazebo>
