Commit message: GPIO

File: sp_description/urdf/test/rmrobot.urdf.xacro (robot description, xacro)
@@ -8,9 +8,9 @@
     <xacro:property name="axel_offset" value="0.05"/> <!-- Space btw top of beam and the each joint -->
     <!-- Used for fixing robot to Gazebo 'base_link' -->
-    <link name="world"/>
+    <!--<link name="world"/>
     <joint name="fixed" type="fixed">
         <parent link="world"/>
         <child link="link1"/>
-    </joint>
+    </joint>-->
     <link name="link1">
         <collision>
@@ -35,8 +35,8 @@
         </inertial>
     </link>
-    <joint name="joint1" type="revolute">
+    <!--<<joint name="joint1" type="revolute">
         <axis xyz="0 1 0"/>
         <origin xyz="0 ${width} ${height1 - axel_offset}" rpy="0 1.57 0"/>
-        <!--      limit not work while type="continuous"-->
+             limit not work while type="continuous"
         <limit effort="5." velocity="50." lower="-1e9" upper="1e9"/>
         <dynamics damping="0.01" friction="0.02"/>
@@ -65,5 +65,5 @@
                     izz="${mass / 12.0 * (width*width + width*width)}"/>
         </inertial>
-    </link>
+    </link>-->
     <transmission name="tran1">
         <type>transmission_interface/SimpleTransmission</type>
@@ -73,5 +73,5 @@
         <actuator name="right_front_wheel_motor">
             <hardwareInterface>hardware_interface/EffortJointInterface</hardwareInterface>
-            <mechanicalReduction>19.20</mechanicalReduction>
+            <mechanicalReduction>1</mechanicalReduction>
         </actuator>
     </transmission>
