Commit message: 更新gpio_controller&修改sp_description路径
1.更新gpio_controller，目的是将其作为基本类型controller使用，具体效果待测
2.为存放新工程模型，更改旧工程模型路径

File: sp_description/urdf/test/rmrobot.xacro (robot description, xacro)
@@ -76,4 +76,14 @@
         </actuator>
     </transmission>
+    <transmission name="tran2">
+        <type>transmission_interface/SimpleTransmission</type>
+        <joint name="joint1">
+            <hardwareInterface>hardware_interface/EffortJointInterface</hardwareInterface>
+        </joint>
+        <actuator name="left_front_wheel_motor">
+            <hardwareInterface>hardware_interface/EffortJointInterface</hardwareInterface>
+            <mechanicalReduction>-1</mechanicalReduction>
+        </actuator>
+    </transmission>
     <gazebo>
         <plugin name="gazebo_ros_control" filename="libgazebo_ros_control.so">
