Commit message: 调整xacro/moveit&新建manipulator类
1.调整xacro配置，新增末端执行link vacuum_gripper
2.调整moveit config
3.manipulator_control下新增Manipulator类管理机械臂运行

File: sp_control/engineer_manipulator_moveit_config/config/gazebo_engineer.urdf (robot description, URDF)
Before this commit: robot engineer, 81 links, 80 joints
Links:
- removed link camera_link
- removed link swiping_card
- added link end_effector_link
- added link link4, mass 0.227354423602744; collision mesh filename=package://sp_description/meshes/engineer_manipulator/link4.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; visual mesh filename=package://sp_description/meshes/engineer_manipulator/link4.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
- added link link5, mass 0.0807348568456161; collision mesh filename=package://sp_description/meshes/engineer_manipulator/link5.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; visual mesh filename=package://sp_description/meshes/engineer_manipulator/link5.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
- added link link6, mass 0.315054913435457; collision mesh filename=package://sp_description/meshes/engineer_manipulator/link6.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; visual mesh filename=package://sp_description/meshes/engineer_manipulator/link6.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
- added link link7, mass 0.226011058027853; collision mesh filename=package://sp_description/meshes/engineer_manipulator/link7.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; visual mesh filename=package://sp_description/meshes/engineer_manipulator/link7.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
- link arm_base_link: mass 0.288208331551669 -> 0.395354400864979; geometry collision mesh filename=package://sp_description/meshes/engineer_manipulator/arm_ba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; visual mesh filename=package://sp_description/meshes/engineer_manipulator/arm_ba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
- link base_link: mass 12.478309558197 -> 10.0515226503987; geometry collision box rpy=0 0 0 size=0.19 0.008 0.12; collision box size=0.144 0.3 0.14
- link fpv_base_link: mass 0.318290775105411 -> 0.317542464634811; geometry collision mesh filename=package://sp_description/meshes/fpv_module/fpv_base_link.STL; visual mesh filename=package://sp_description/meshes/fpv_module/fpv_base_link.STL
- link fpv_pitch: mass 0.790822100365449 -> 0.79082; geometry collision mesh filename=package://sp_description/meshes/fpv_module/fpv_pitch.STL; visual mesh filename=package://sp_description/meshes/fpv_module/fpv_pitch.STL
- link fpv_yaw: mass 0.0608808554843221 -> 0.060612; geometry collision mesh filename=package://sp_description/meshes/fpv_module/fpv_yaw.STL; visual mesh filename=package://sp_description/meshes/fpv_module/fpv_yaw.STL
- link left_back_wheel: mass 0.59 -> 0.4235; geometry visual mesh filename=package://sp_description/meshes/common/mecanum_wheel/left_m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
- link left_front_wheel: mass 0.59 -> 0.4235; geometry visual mesh filename=package://sp_description/meshes/common/mecanum_wheel/right_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
- link link1: mass 0.378634616635792 -> 0.376683384729688; geometry collision mesh filename=package://sp_description/meshes/engineer_manipulator/link1.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; visual mesh filename=package://sp_description/meshes/engineer_manipulator/link1.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
- link link2: mass 0.992951364752065 -> 0.759246586931641; geometry collision mesh filename=package://sp_description/meshes/engineer_manipulator/link2.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; visual mesh filename=package://sp_description/meshes/engineer_manipulator/link2.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
- link link3: mass 1.29043542087694 -> 0.728531979995667; geometry collision mesh filename=package://sp_description/meshes/engineer_manipulator/link3.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; visual mesh filename=package://sp_description/meshes/engineer_manipulator/link3.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
- link mast: mass 0.434967907171886 -> 0.596769834435929; geometry collision mesh filename=package://sp_description/meshes/fpv_module/mast.STL; visual mesh filename=package://sp_description/meshes/fpv_module/mast.STL
- link right_back_wheel: mass 0.59 -> 0.4235; geometry visual mesh filename=package://sp_description/meshes/common/mecanum_wheel/right_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
- link right_front_wheel: mass 0.59 -> 0.4235; geometry visual mesh filename=package://sp_description/meshes/common/mecanum_wheel/left_m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
Joints:
- removed joint camera_joint
- removed joint card_joint
- added joint end_effector_joint: type fixed, parent link7, child end_effector_link, origin xyz=0 0 0.054 rpy=0 0 0, axis 0 0 1
- added joint joint4: type revolute, parent link3, child link4, origin xyz=0.13435 0 0 rpy=0 1.5708 0, axis 0 0 1, limit lower=-3.14 upper=3.14 effort=20 velocity=5
- added joint joint5: type revolute, parent link4, child link5, origin xyz=0 -0.025 0.05 rpy=1.5708 -1.5708 0, axis 0 0 -1, limit lower=-1.90 upper=1.57 effort=20 velocity=5
- added joint joint6: type revolute, parent link5, child link6, origin xyz=0.091 0 -0.025 rpy=-1.5708 0 -1.5708, axis 0 0 1, limit lower=-3.14 upper=3.14 effort=20 velocity=5
- added joint joint7: type prismatic, parent link6, child link7, origin xyz=0 0 0.02445 rpy=0 0 0, axis 0 0 -1, limit lower=-0.075 upper=0 effort=20 velocity=5
- joint fpv_pitch_joint: origin xyz=0 0.0007 0.0275 rpy=-1.5708 0 -3.1416 -> xyz=0 0.000700000000000704 0.0275 rpy=-1.5707963267949 0 3.14159265358979
- joint joint1: origin xyz=0 0 0.024 rpy=0 0 0 -> xyz=0 0 0 rpy=0 0 0
- joint joint2: origin xyz=0 0.022 0.065 rpy=1.5708 -1.5708 0 -> xyz=-0.022 0 0.065 rpy=0 -1.5708 0
- joint joint3: axis 0 0 -1 -> 0 0 1; origin xyz=0.199986932336027 0.00228624032540565 0 rpy=0 0 0.0114314489445579 -> xyz=0.2 0 0 rpy=0 0 0
- joint joint_arm2body: origin xyz=0.0445 0.197 0.237 rpy=0 0 0 -> xyz=0.022 0.166 0.228 rpy=0 0 -1.5708
- joint joint_mast2body: origin xyz=-0.2295 -0.0815 0.0157 rpy=0 0 1.5707 -> xyz=-0.2295 -0.0825 0.0177 rpy=0 0 1.5708
- joint left_back_roller_0_joint: origin xyz=4.117874862132975e-18 0 -0.06725 rpy=0 0 0 -> xyz=4.163799117101001e-18 0 -0.068 rpy=0 0 0
- joint left_back_roller_10_joint: origin xyz=-0.04769581099104322 0 0.04740962047840798 rpy=0 0 0 -> xyz=-0.048227734533694264 0 0.04793835230530472 rpy=0 0 0
- joint left_back_roller_11_joint: origin xyz=-0.06221574501182705 0 0.02552966064449972 rpy=0 0 0 -> xyz=-0.06290960090415226 0 0.02581437804945697 rpy=0 0 0
- joint left_back_roller_12_joint: origin xyz=-0.06724956154854442 0 -0.00024284054137712588 rpy=0 0 0 -> xyz=-0.06799955665875124 0 -0.0002455488002028931 rpy=0 0 0
- joint left_back_roller_13_joint: origin xyz=-0.062029747891165755 0 -0.025978315506560806 rpy=0 0 0 -> xyz=-0.06272152946616016 0 -0.026268036497340295 rpy=0 0 0
- joint left_back_roller_14_joint: origin xyz=-0.047352175978368535 0 -0.04775284211556018 rpy=0 0 0 -> xyz=-0.04788026716028342 0 -0.04828540169305713 rpy=0 0 0
- joint left_back_roller_15_joint: origin xyz=-0.025454754743320145 0 -0.06224642930287183 rpy=0 0 0 -> xyz=-0.025738636766479847 0 -0.06294062739918639 rpy=0 0 0
- joint left_back_roller_1_joint: origin xyz=0.025754155985525513 0 -0.06212315147731336 rpy=0 0 0 -> xyz=0.026041377055996056 0 -0.06281597472798972 rpy=0 0 0
- joint left_back_roller_2_joint: origin xyz=0.04758154151551398 0 -0.04752430333005861 rpy=0 0 0 -> xyz=0.04811219067739703 0 -0.048054314147865956 rpy=0 0 0
- joint left_back_roller_3_joint: origin xyz=0.062154106054395655 0 -0.02567936137404779 rpy=0 0 0 -> xyz=0.06284727452340379 0 -0.025965748303869884 rpy=0 0 0
- joint left_back_roller_4_joint: origin xyz=0.06724995128312455 0 8.094700349681064e-05 rpy=0 0 0 -> xyz=0.06799995073981367 0 8.184975818264867e-05 rpy=0 0 0
- joint left_back_roller_5_joint: origin xyz=0.06209210689440703 0 0.025828913283634913 rpy=0 0 0 -> xyz=0.06278458392296919 0 0.026116968078619688 rpy=0 0 0
- joint left_back_roller_6_joint: origin xyz=0.04746699629001391 0 0.04763871076345167 rpy=0 0 0 -> xyz=0.0479963679958505 0 0.04816999750059053 rpy=0 0 0
- joint left_back_roller_7_joint: origin xyz=0.02560452955756635 0 0.06218497058080603 rpy=0 0 0 -> xyz=0.0258900819318143 0 0.06287848326386335 rpy=0 0 0
- joint left_back_roller_8_joint: origin xyz=-0.0001618938897152502 0 0.06724980513256877 rpy=0 0 0 -> xyz=-0.00016369939777898906 0 0.06799980295932605 rpy=0 0 0
- joint left_back_roller_9_joint: origin xyz=-0.025903633160065442 0 0.062060972350654955 rpy=0 0 0 -> xyz=-0.026192521262222306 0 0.06275310215382211 rpy=0 0 0
- joint left_back_wheel_joint: origin xyz=-0.19727 0.223 -0.00111 rpy=0 0 0 -> xyz=-0.19727 0.223 0.000889 rpy=0 0 0
- joint left_front_roller_0_joint: origin xyz=4.117874862132975e-18 0 -0.06725 rpy=0 0 0 -> xyz=4.163799117101001e-18 0 -0.068 rpy=0 0 0
- joint left_front_roller_10_joint: origin xyz=-0.04769581099104322 0 0.04740962047840798 rpy=0 0 0 -> xyz=-0.048227734533694264 0 0.04793835230530472 rpy=0 0 0
- joint left_front_roller_11_joint: origin xyz=-0.06221574501182705 0 0.02552966064449972 rpy=0 0 0 -> xyz=-0.06290960090415226 0 0.02581437804945697 rpy=0 0 0
- joint left_front_roller_12_joint: origin xyz=-0.06724956154854442 0 -0.00024284054137712588 rpy=0 0 0 -> xyz=-0.06799955665875124 0 -0.0002455488002028931 rpy=0 0 0
- joint left_front_roller_13_joint: origin xyz=-0.062029747891165755 0 -0.025978315506560806 rpy=0 0 0 -> xyz=-0.06272152946616016 0 -0.026268036497340295 rpy=0 0 0
- joint left_front_roller_14_joint: origin xyz=-0.047352175978368535 0 -0.04775284211556018 rpy=0 0 0 -> xyz=-0.04788026716028342 0 -0.04828540169305713 rpy=0 0 0
- joint left_front_roller_15_joint: origin xyz=-0.025454754743320145 0 -0.06224642930287183 rpy=0 0 0 -> xyz=-0.025738636766479847 0 -0.06294062739918639 rpy=0 0 0
- joint left_front_roller_1_joint: origin xyz=0.025754155985525513 0 -0.06212315147731336 rpy=0 0 0 -> xyz=0.026041377055996056 0 -0.06281597472798972 rpy=0 0 0
- joint left_front_roller_2_joint: origin xyz=0.04758154151551398 0 -0.04752430333005861 rpy=0 0 0 -> xyz=0.04811219067739703 0 -0.048054314147865956 rpy=0 0 0
- joint left_front_roller_3_joint: origin xyz=0.062154106054395655 0 -0.02567936137404779 rpy=0 0 0 -> xyz=0.06284727452340379 0 -0.025965748303869884 rpy=0 0 0
- joint left_front_roller_4_joint: origin xyz=0.06724995128312455 0 8.094700349681064e-05 rpy=0 0 0 -> xyz=0.06799995073981367 0 8.184975818264867e-05 rpy=0 0 0
- joint left_front_roller_5_joint: origin xyz=0.06209210689440703 0 0.025828913283634913 rpy=0 0 0 -> xyz=0.06278458392296919 0 0.026116968078619688 rpy=0 0 0
- joint left_front_roller_6_joint: origin xyz=0.04746699629001391 0 0.04763871076345167 rpy=0 0 0 -> xyz=0.0479963679958505 0 0.04816999750059053 rpy=0 0 0
- joint left_front_roller_7_joint: origin xyz=0.02560452955756635 0 0.06218497058080603 rpy=0 0 0 -> xyz=0.0258900819318143 0 0.06287848326386335 rpy=0 0 0
- joint left_front_roller_8_joint: origin xyz=-0.0001618938897152502 0 0.06724980513256877 rpy=0 0 0 -> xyz=-0.00016369939777898906 0 0.06799980295932605 rpy=0 0 0
- joint left_front_roller_9_joint: origin xyz=-0.025903633160065442 0 0.062060972350654955 rpy=0 0 0 -> xyz=-0.026192521262222306 0 0.06275310215382211 rpy=0 0 0
- joint left_front_wheel_joint: origin xyz=0.19727 0.223 -0.00111 rpy=0 0 0 -> xyz=0.19727 0.223 0.000889 rpy=0 0 0
- joint right_back_roller_0_joint: origin xyz=4.117874862132975e-18 0 -0.06725 rpy=0 0 0 -> xyz=4.163799117101001e-18 0 -0.068 rpy=0 0 0
- joint right_back_roller_10_joint: origin xyz=-0.04769581099104322 0 0.04740962047840798 rpy=0 0 0 -> xyz=-0.048227734533694264 0 0.04793835230530472 rpy=0 0 0
- joint right_back_roller_11_joint: origin xyz=-0.06221574501182705 0 0.02552966064449972 rpy=0 0 0 -> xyz=-0.06290960090415226 0 0.02581437804945697 rpy=0 0 0
- joint right_back_roller_12_joint: origin xyz=-0.06724956154854442 0 -0.00024284054137712588 rpy=0 0 0 -> xyz=-0.06799955665875124 0 -0.0002455488002028931 rpy=0 0 0
- joint right_back_roller_13_joint: origin xyz=-0.062029747891165755 0 -0.025978315506560806 rpy=0 0 0 -> xyz=-0.06272152946616016 0 -0.026268036497340295 rpy=0 0 0
- joint right_back_roller_14_joint: origin xyz=-0.047352175978368535 0 -0.04775284211556018 rpy=0 0 0 -> xyz=-0.04788026716028342 0 -0.04828540169305713 rpy=0 0 0
- joint right_back_roller_15_joint: origin xyz=-0.025454754743320145 0 -0.06224642930287183 rpy=0 0 0 -> xyz=-0.025738636766479847 0 -0.06294062739918639 rpy=0 0 0
- joint right_back_roller_1_joint: origin xyz=0.025754155985525513 0 -0.06212315147731336 rpy=0 0 0 -> xyz=0.026041377055996056 0 -0.06281597472798972 rpy=0 0 0
- joint right_back_roller_2_joint: origin xyz=0.04758154151551398 0 -0.04752430333005861 rpy=0 0 0 -> xyz=0.04811219067739703 0 -0.048054314147865956 rpy=0 0 0
- joint right_back_roller_3_joint: origin xyz=0.062154106054395655 0 -0.02567936137404779 rpy=0 0 0 -> xyz=0.06284727452340379 0 -0.025965748303869884 rpy=0 0 0
- joint right_back_roller_4_joint: origin xyz=0.06724995128312455 0 8.094700349681064e-05 rpy=0 0 0 -> xyz=0.06799995073981367 0 8.184975818264867e-05 rpy=0 0 0
- joint right_back_roller_5_joint: origin xyz=0.06209210689440703 0 0.025828913283634913 rpy=0 0 0 -> xyz=0.06278458392296919 0 0.026116968078619688 rpy=0 0 0
- joint right_back_roller_6_joint: origin xyz=0.04746699629001391 0 0.04763871076345167 rpy=0 0 0 -> xyz=0.0479963679958505 0 0.04816999750059053 rpy=0 0 0
- joint right_back_roller_7_joint: origin xyz=0.02560452955756635 0 0.06218497058080603 rpy=0 0 0 -> xyz=0.0258900819318143 0 0.06287848326386335 rpy=0 0 0
- joint right_back_roller_8_joint: origin xyz=-0.0001618938897152502 0 0.06724980513256877 rpy=0 0 0 -> xyz=-0.00016369939777898906 0 0.06799980295932605 rpy=0 0 0
- joint right_back_roller_9_joint: origin xyz=-0.025903633160065442 0 0.062060972350654955 rpy=0 0 0 -> xyz=-0.026192521262222306 0 0.06275310215382211 rpy=0 0 0
- joint right_back_wheel_joint: origin xyz=-0.19727 -0.223 -0.00111 rpy=0 0 0 -> xyz=-0.19727 -0.223 0.000889 rpy=0 0 0
- joint right_front_roller_0_joint: origin xyz=4.117874862132975e-18 0 -0.06725 rpy=0 0 0 -> xyz=4.163799117101001e-18 0 -0.068 rpy=0 0 0
- joint right_front_roller_10_joint: origin xyz=-0.04769581099104322 0 0.04740962047840798 rpy=0 0 0 -> xyz=-0.048227734533694264 0 0.04793835230530472 rpy=0 0 0
- joint right_front_roller_11_joint: origin xyz=-0.06221574501182705 0 0.02552966064449972 rpy=0 0 0 -> xyz=-0.06290960090415226 0 0.02581437804945697 rpy=0 0 0
- joint right_front_roller_12_joint: origin xyz=-0.06724956154854442 0 -0.00024284054137712588 rpy=0 0 0 -> xyz=-0.06799955665875124 0 -0.0002455488002028931 rpy=0 0 0
- joint right_front_roller_13_joint: origin xyz=-0.062029747891165755 0 -0.025978315506560806 rpy=0 0 0 -> xyz=-0.06272152946616016 0 -0.026268036497340295 rpy=0 0 0
- joint right_front_roller_14_joint: origin xyz=-0.047352175978368535 0 -0.04775284211556018 rpy=0 0 0 -> xyz=-0.04788026716028342 0 -0.04828540169305713 rpy=0 0 0
- joint right_front_roller_15_joint: origin xyz=-0.025454754743320145 0 -0.06224642930287183 rpy=0 0 0 -> xyz=-0.025738636766479847 0 -0.06294062739918639 rpy=0 0 0
- joint right_front_roller_1_joint: origin xyz=0.025754155985525513 0 -0.06212315147731336 rpy=0 0 0 -> xyz=0.026041377055996056 0 -0.06281597472798972 rpy=0 0 0
- joint right_front_roller_2_joint: origin xyz=0.04758154151551398 0 -0.04752430333005861 rpy=0 0 0 -> xyz=0.04811219067739703 0 -0.048054314147865956 rpy=0 0 0
- joint right_front_roller_3_joint: origin xyz=0.062154106054395655 0 -0.02567936137404779 rpy=0 0 0 -> xyz=0.06284727452340379 0 -0.025965748303869884 rpy=0 0 0
- joint right_front_roller_4_joint: origin xyz=0.06724995128312455 0 8.094700349681064e-05 rpy=0 0 0 -> xyz=0.06799995073981367 0 8.184975818264867e-05 rpy=0 0 0
- joint right_front_roller_5_joint: origin xyz=0.06209210689440703 0 0.025828913283634913 rpy=0 0 0 -> xyz=0.06278458392296919 0 0.026116968078619688 rpy=0 0 0
- joint right_front_roller_6_joint: origin xyz=0.04746699629001391 0 0.04763871076345167 rpy=0 0 0 -> xyz=0.0479963679958505 0 0.04816999750059053 rpy=0 0 0
- joint right_front_roller_7_joint: origin xyz=0.02560452955756635 0 0.06218497058080603 rpy=0 0 0 -> xyz=0.0258900819318143 0 0.06287848326386335 rpy=0 0 0
- joint right_front_roller_8_joint: origin xyz=-0.0001618938897152502 0 0.06724980513256877 rpy=0 0 0 -> xyz=-0.00016369939777898906 0 0.06799980295932605 rpy=0 0 0
- joint right_front_roller_9_joint: origin xyz=-0.025903633160065442 0 0.062060972350654955 rpy=0 0 0 -> xyz=-0.026192521262222306 0 0.06275310215382211 rpy=0 0 0
- joint right_front_wheel_joint: origin xyz=0.19727 -0.223 -0.00111 rpy=0 0 0 -> xyz=0.19727 -0.223 0.000889 rpy=0 0 0
- joint rplidar_back_joint: origin xyz=-0.22 0 0.165 rpy=0 0 3.14159 -> xyz=-0.22 0 0.165 rpy=0 0 3.1416

File: sp_description/urdf/engineer/engineer.xacro (robot description, xacro)
@@ -1,24 +1,13 @@
 <?xml version="1.0"?>
 <robot xmlns:xacro="http://www.ros.org/wiki/xacro" name="engineer">
-	<xacro:include filename="$(find sp_description)/urdf/engineer/engineer2_manipulator/manipulator_test.xacro"/>
+	<xacro:include filename="$(find sp_description)/urdf/engineer/engineer_manipulator/engineer_manipulator.xacro"/>
 	<xacro:include filename="$(find sp_description)/urdf/engineer/engineer_chassis/engineer_chassis.xacro"/>
-<<<<<<< Updated upstream
 	<xacro:include filename="$(find sp_description)/urdf/engineer/manipulator_transmission.xacro"/>
 	<xacro:include filename="$(find sp_description)/urdf/engineer/fpv_module/fpv_module.xacro"/>
 	<xacro:include filename="$(find sp_description)/urdf/common/lidar2d.xacro"/>
-=======
-	<xacro:include filename="$(find sp_description)/urdf/engineer/manipulator_transmission_test.xacro"/>
-	<xacro:include filename="$(find sp_description)/urdf/engineer/fpv_module/fpv_module_test.xacro"/>
-	<xacro:include filename="$(find sp_description)/urdf/common/lidar2d.urdf.xacro"/>
->>>>>>> Stashed changes
 	<xacro:arg name="use_simulation" default="true"/>
 	<xacro:engineer_chassis roller_type="simple"/>
 	<xacro:fpv_module/>
-<<<<<<< Updated upstream
 	<xacro:engineer_manipulator/>
-=======
-	<xacro:engineer2_manipulator/>
-	<xacro:swiping_card />
->>>>>>> Stashed changes
 	<xacro:lidar2d connected_to="base_link" lidar_name="rplidar_front"
 				   simulation="$(arg use_simulation)"

File: sp_description/urdf/engineer/engineer_chassis/engineer_chassis.xacro (robot description, xacro)
@@ -49,5 +49,5 @@
       <origin xyz="0 0 0" rpy="0 0 0" />
       <geometry>
-        <box size="0.6 0.6 0.15"/>
+        <box size="0.6 0.6 0.150"/>
       </geometry>
     </collision>
@@ -83,13 +83,13 @@
     </collision>
     <collision>
-      <origin xyz="0.0 0.054 0.23" rpy="0 0 0"/>
-      <geometry>
-        <box size="0.19 0.008 0.12" rpy="0 0 0"/>
-      </geometry>
-    </collision>
-    <collision>
-      <origin xyz="0.0 -0.172 0.23" rpy="0 0 0"/>
-      <geometry>
-        <box size="0.19 0.01 0.12"/>
+      <origin xyz="0.0 0.054 0.10" rpy="0 0 0"/>
+      <geometry>
+        <box size="0.19 0.008 0.10" rpy="0 0 0"/>
+      </geometry>
+    </collision>
+    <collision>
+      <origin xyz="0.0 -0.172 0.10" rpy="0 0 0"/>
+      <geometry>
+        <box size="0.19 0.01 0.10"/>
       </geometry>
     </collision>

File: sp_description/urdf/engineer/engineer_manipulator/engineer_manipulator.xacro (robot description, xacro)
@@ -214,6 +214,6 @@
         xyz="0 0 1" />
       <limit
-        lower="-1.57"
-        upper="1.57"
+        lower="-1.80"
+        upper="1.80"
         effort="20"
         velocity="5" />
@@ -330,5 +330,5 @@
         xyz="0 0 -1" />
       <limit
-        lower="-1.57"
+        lower="-1.90"
         upper="1.57"
         effort="20"
@@ -446,8 +446,22 @@
         xyz="0 0 -1" />
       <limit
-        lower="-0.11"
+        lower="-0.075"
         upper="0"
         effort="20"
         velocity="5" />
+    </joint>
+    <link name="vacuum_gripper"/>
+    <joint
+      name="vacuum_gripper_joint"
+      type="fixed">
+      <origin
+        xyz="0 0 0.054"
+        rpy="0 0 0" />
+      <parent
+        link="link7" />
+      <child
+        link="vacuum_gripper" />
+      <axis
+        xyz="0 0 1" />
     </joint>
   </xacro:macro>

File: sp_description/urdf/engineer/manipulator_transmission.xacro (robot description, xacro)
@@ -1,4 +1,4 @@
 <?xml version="1.0" encoding="utf-8"?>
-<robot xmlns:xacro="http://www.ros.org/wiki/xacro" name="engineer2_manipulator">
+<robot xmlns:xacro="http://www.ros.org/wiki/xacro" name="engineer_manipulator">
     <xacro:macro name="manipulator_transmission" params="joint_name">
         <transmission name="trans_${joint_name}">
@@ -20,3 +20,23 @@
     <xacro:manipulator_transmission joint_name="joint6"/>
     <xacro:manipulator_transmission joint_name="joint7"/>
+    <gazebo>
+        <plugin name="gazebo_ros_vacuum_gripper" filename="libgazebo_ros_vacuum_gripper.so">
+            <robotNamespace>/vacuum_gripper</robotNamespace>
+            <bodyName>vacuum_gripper</bodyName>
+            <topicName>grasping</topicName>
+            <maxForce>100</maxForce>
+            <maxDistance>0.05</maxDistance>
+            <minDistance>0.01</minDistance>
+        </plugin>
+    </gazebo>
+    <gazebo reference="vacuum_gripper">
+        <mu1>50</mu1>
+        <mu2>50</mu2>
+　　　   <minDepth>0.003</minDepth>
+        <maxVel>0</maxVel>
+        <kp>10000000000000.0</kp>
+        <kd>1.0</kd>
+        <ki>2.0</ki>
+        <material>Gazebo/Grey</material>
+    </gazebo>
 </robot>

File: sp_description/urdf/test/rmrobot.urdf.xacro (robot description, xacro)
@@ -73,5 +73,5 @@
         <actuator name="right_front_wheel_motor">
             <hardwareInterface>hardware_interface/EffortJointInterface</hardwareInterface>
-            <mechanicalReduction>6</mechanicalReduction>
+            <mechanicalReduction>19.2032</mechanicalReduction>
         </actuator>
     </transmission>
