Commit message: update sp_hw,etc

File: sp_control/engineer_manipulator_moveit_config/config/gazebo_engineer.urdf (robot description, URDF)
Before this commit: robot engineer, 84 links, 83 joints
Links:
- removed link end_effector_link
- removed link rplidar_back
- removed link rplidar_front
- added link vacuum_gripper
- link base_link: geometry collision box rpy=0 0 0 size=0.19 0.008 0.10; collision box size=0.144 0.3 0.14
- link link6: mass 0.315054913435457 -> 0.25692
- link link7: mass 0.226011058027853 -> 0.20296
Joints:
- removed joint end_effector_joint
- removed joint rplidar_back_joint
- removed joint rplidar_front_joint
- added joint vacuum_gripper_joint: type fixed, parent link7, child vacuum_gripper, origin xyz=0 0 0.054 rpy=0 0 0, axis 0 0 1
- joint fpv_yaw_joint: origin xyz=0 -0.0285 0.3853 rpy=0 0 0 -> xyz=0 -0.0285 0.3853 rpy=0 0 -1.5707963267949
- joint joint2: axis 0 0 -1 -> 0 0 1; limit lower=-1.57 upper=1.57 effort=20 velocity=5 -> lower=-1.70 upper=1.70 effort=20 velocity=5
- joint joint3: axis 0 0 1 -> 0 0 -1; limit lower=-1.57 upper=1.57 effort=20 velocity=5 -> lower=-2.80 upper=2.80 effort=20 velocity=5
- joint joint5: axis 0 0 -1 -> 0 0 1; limit lower=-1.90 upper=1.57 effort=20 velocity=5 -> lower=-2.10 upper=2.10 effort=20 velocity=5
- joint joint6: limit lower=-3.14 upper=3.14 effort=20 velocity=5 -> lower=-1.57 upper=1.57 effort=20 velocity=5; origin xyz=0.091 0 -0.025 rpy=-1.5708 0 -1.5708 -> xyz=0.096 0 -0.03 rpy=-1.5708 0.05753 -1.5708
- joint joint7: origin xyz=0 0 0.02445 rpy=0 0 0 -> xyz=0 0 0.025373 rpy=0 0 0

File: sp_description/urdf/engineer/engineer.xacro (robot description, xacro)
@@ -3,10 +3,12 @@
 	<xacro:include filename="$(find sp_description)/urdf/engineer/engineer_manipulator/engineer_manipulator.xacro"/>
 	<xacro:include filename="$(find sp_description)/urdf/engineer/engineer_chassis/engineer_chassis.xacro"/>
-	<xacro:include filename="$(find sp_description)/urdf/engineer/manipulator_transmission.xacro"/>
+	<!--<xacro:include filename="$(find sp_description)/urdf/engineer/manipulator_transmission.xacro"/>
 	<xacro:include filename="$(find sp_description)/urdf/engineer/fpv_module/fpv_module.xacro"/>
+-->
 	<xacro:arg name="use_simulation" default="true"/>
 	<xacro:engineer_chassis roller_type="simple"/>
-	<xacro:fpv_module/>
-	<xacro:engineer_manipulator/>
+	<!--<xacro:fpv_module/>
+	<xacro:engineer_manipulator/>-->
+<!--
 	<joint name="joint_arm2body" type="fixed">
 		<axis xyz="0 0 1"/>
@@ -20,5 +22,5 @@
 			<parent link="base_link"/>
 			<child link="fpv_base_link"/>
-	</joint>
+	</joint>-->
 	<gazebo>
 		<plugin name="gazebo_ros_control" filename="libgazebo_ros_control.so">

File: sp_description/urdf/engineer/engineer_manipulator/engineer_manipulator.xacro (robot description, xacro)
@@ -456,5 +456,5 @@
       type="fixed">
       <origin
-        xyz="0 0 0.054"
+        xyz="0 0 0.048"
         rpy="0 0 0" />
       <parent

File: sp_description/urdf/engineer/fpv_module/fpv_module.xacro (robot description, xacro)
@@ -98,5 +98,5 @@
       link="mast" />
     <axis
-      xyz="0 0 1" />
+      xyz="0 0 -1" />
     <limit
       lower="0"
@@ -225,8 +225,8 @@
     <type>transmission_interface/SimpleTransmission</type>
     <actuator name="mast_joint_motor">
-      <mechanicalReduction>1</mechanicalReduction>
+      <mechanicalReduction>50</mechanicalReduction>
     </actuator>
     <joint name="mast_joint">
-      <hardwareInterface>hardware_interface/PositionJointInterface</hardwareInterface>
+      <hardwareInterface>hardware_interface/EffortJointInterface</hardwareInterface>
     </joint>
   </transmission>

File: sp_description/urdf/engineer/manipulator_transmission.xacro (robot description, xacro)
@@ -6,8 +6,8 @@
             <actuator name="${joint_name}_motor">
                 <mechanicalReduction>${mechanical_reduction}</mechanicalReduction>
-				<hardwareInterface>hardware_interface/PositionJointInterface</hardwareInterface>
+				<hardwareInterface>hardware_interface/EffortJointInterface</hardwareInterface>
             </actuator>
 			<joint name="${joint_name}">
-				<hardwareInterface>hardware_interface/PositionJointInterface</hardwareInterface>
+				<hardwareInterface>hardware_interface/EffortJointInterface</hardwareInterface>
 			</joint>
         </transmission>

Commit message: 微调xacro等

File: sp_control/engineer_manipulator_moveit_config/config/gazebo_engineer.urdf (robot description, URDF)
Before this commit: robot engineer, 82 links, 81 joints
Links:
- link arm_base_link: geometry collision mesh filename=package://sp_description/meshes/engineer_manipulator/engine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; visual mesh filename=package://sp_description/meshes/engineer_manipulator/engine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
- link base_link: geometry collision box rpy=0 0 0 size=0.19 0.008 0.10; collision box size=0.144 0.3 0.14
- link fpv_base_link: geometry collision mesh filename=package://sp_description/meshes/engineer_manipulator/fpv_mo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; visual mesh filename=package://sp_description/meshes/engineer_manipulator/fpv_mo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
- link fpv_pitch: geometry collision mesh filename=package://sp_description/meshes/engineer_manipulator/fpv_mo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; visual mesh filename=package://sp_description/meshes/engineer_manipulator/fpv_mo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
- link fpv_yaw: geometry collision mesh filename=package://sp_description/meshes/engineer_manipulator/fpv_mo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; visual mesh filename=package://sp_description/meshes/engineer_manipulator/fpv_mo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
- link link1: geometry collision mesh filename=package://sp_description/meshes/engineer_manipulator/engine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; visual mesh filename=package://sp_description/meshes/engineer_manipulator/engine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
- link link2: geometry collision mesh filename=package://sp_description/meshes/engineer_manipulator/engine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; visual mesh filename=package://sp_description/meshes/engineer_manipulator/engine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
- link link3: geometry collision mesh filename=package://sp_description/meshes/engineer_manipulator/engine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; visual mesh filename=package://sp_description/meshes/engineer_manipulator/engine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
- link link4: geometry collision mesh filename=package://sp_description/meshes/engineer_manipulator/engine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; visual mesh filename=package://sp_description/meshes/engineer_manipulator/engine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
- link link5: geometry collision mesh filename=package://sp_description/meshes/engineer_manipulator/engine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; visual mesh filename=package://sp_description/meshes/engineer_manipulator/engine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
- link link6: geometry collision mesh filename=package://sp_description/meshes/engineer_manipulator/engine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; visual mesh filename=package://sp_description/meshes/engineer_manipulator/engine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
- link link7: geometry collision mesh filename=package://sp_description/meshes/engineer_manipulator/engine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; visual mesh filename=package://sp_description/meshes/engineer_manipulator/engine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
- link mast: geometry collision mesh filename=package://sp_description/meshes/engineer_manipulator/fpv_mo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; visual mesh filename=package://sp_description/meshes/engineer_manipulator/fpv_mo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
Joints:
- joint fpv_yaw_joint: limit lower=-1.5708 upper=1.5708 effort=1.3 velocity=6 -> lower=-1.80 upper=1.50 effort=1.3 velocity=6
- joint joint1: limit lower=-3.14 upper=3.14 effort=20 velocity=5 -> lower=-3.14 upper=3.14 effort=20 velocity=6
- joint joint2: limit lower=-1.70 upper=1.70 effort=20 velocity=5 -> lower=-1.70 upper=1.70 effort=20 velocity=8
- joint joint3: limit lower=-2.80 upper=2.80 effort=20 velocity=5 -> lower=-2.80 upper=2.80 effort=20 velocity=8
- joint joint4: limit lower=-3.14 upper=3.14 effort=20 velocity=5 -> lower=-3.14 upper=3.14 effort=20 velocity=7
- joint joint5: limit lower=-2.10 upper=2.10 effort=20 velocity=5 -> lower=-2.10 upper=2.10 effort=20 velocity=7
- joint joint6: limit lower=-1.57 upper=1.57 effort=20 velocity=5 -> lower=-3.14 upper=3.14 effort=20 velocity=7
- joint joint7: limit lower=-0.075 upper=0 effort=20 velocity=5 -> lower=-0.075 upper=0 effort=20 velocity=0.075
- joint mast_joint: axis 0 0 1 -> 0 0 -1; limit lower=0 upper=0.235 effort=50 velocity=0.8 -> lower=-0.235 upper=0 effort=50 velocity=0.4
- joint vacuum_gripper_joint: origin xyz=0 0 0.054 rpy=0 0 0 -> xyz=0 0 0.055 rpy=0 0 0

File: sp_description/urdf/engineer_manipulator/engineer.xacro (robot description, xacro)
@@ -1,5 +1,5 @@
 <?xml version="1.0"?>
 <robot xmlns:xacro="http://www.ros.org/wiki/xacro" name="engineer">
-	<xacro:include filename="$(find sp_description)/urdf/engineer_manipulator/engineer_manipulator/engineer_manipulator.xacro"/>
+    <xacro:include filename="$(find sp_description)/urdf/engineer_manipulator/engineer_manipulator/engineer_manipulator.xacro"/>
 	<xacro:include filename="$(find sp_description)/urdf/engineer_manipulator/engineer_chassis/engineer_chassis.xacro"/>
 	<xacro:include filename="$(find sp_description)/urdf/engineer_manipulator/manipulator_transmission.xacro"/>
@@ -9,5 +9,5 @@
 	<xacro:fpv_module/>
 	<xacro:engineer_manipulator/>
-	<joint name="joint_arm2body" type="fixed">
+<joint name="joint_arm2body" type="fixed">
 		<axis xyz="0 0 1"/>
 		<origin xyz="0.022 0.166 0.228" rpy="0 0 -1.5708"/>

File: sp_description/urdf/engineer_manipulator/engineer_chassis/engineer_chassis.xacro (robot description, xacro)
@@ -111,8 +111,8 @@
                          wheel_z_offset="${wheel_offset_z}"
                          reflect="1" roller_type="${roller_type}"/>
-    <xacro:wheel_transmission prefix="left_front" mechanical_reduction="19.2032"/>
-    <xacro:wheel_transmission prefix="right_front" mechanical_reduction="-19.2032"/>
-    <xacro:wheel_transmission prefix="left_back" mechanical_reduction="19.2032"/>
-    <xacro:wheel_transmission prefix="right_back" mechanical_reduction="-19.2032"/>
+    <xacro:wheel_transmission prefix="left_front" mechanical_reduction="1"/>
+    <xacro:wheel_transmission prefix="right_front" mechanical_reduction="-1"/>
+    <xacro:wheel_transmission prefix="left_back" mechanical_reduction="1"/>
+    <xacro:wheel_transmission prefix="right_back" mechanical_reduction="-1"/>
   </xacro:macro>
 `

File: sp_description/urdf/engineer_manipulator/engineer_manipulator/engineer_manipulator.xacro (robot description, xacro)
@@ -32,5 +32,5 @@
           name="">
           <color
-            rgba="0.333333333333333 0.333333333333333 0.333333333333333 1" />
+            rgba="1 1 1 1" />
         </material>
       </visual>
@@ -72,5 +72,5 @@
           name="">
           <color
-            rgba="0.333333333333333 0.333333333333333 0.333333333333333 1" />
+            rgba="1 1 1 1" />
         </material>
       </visual>
@@ -130,5 +130,5 @@
           name="">
           <color
-            rgba="0.333333333333333 0.333333333333333 0.333333333333333 1" />
+            rgba="1 1 1 1" />
         </material>
       </visual>
@@ -188,5 +188,5 @@
           name="">
           <color
-            rgba="0.333333333333333 0.333333333333333 0.333333333333333 1" />
+            rgba="1 1 1 1" />
         </material>
       </visual>
@@ -246,5 +246,5 @@
           name="">
           <color
-            rgba="0.823529411764706 0.870588235294118 0.980392156862745 1" />
+            rgba="1 1 1 1" />
         </material>
       </visual>
@@ -304,5 +304,5 @@
           name="">
           <color
-            rgba="0.792156862745098 0.819607843137255 0.933333333333333 1" />
+            rgba="1 1 1 1" />
         </material>
       </visual>
@@ -362,5 +362,5 @@
         name="">
         <color
-          rgba="0.49804 0.49804 0.49804 1" />
+          rgba="1 1 1 1" />
       </material>
     </visual>
@@ -420,5 +420,5 @@
         name="">
         <color
-          rgba="0.33333 0.33333 0.33333 1" />
+          rgba="1 1 1 1" />
       </material>
     </visual>

File: sp_description/urdf/test/rmrobot.xacro (robot description, xacro)
@@ -35,5 +35,5 @@
         </inertial>
     </link>
-    <joint name="joint1" type="prismatic">
+    <joint name="joint1" type="revolute">
         <axis xyz="0 1 0"/>
         <origin xyz="0 ${width} ${height1 - axel_offset}" rpy="0 1.57 0"/>
@@ -73,15 +73,5 @@
         <actuator name="right_front_wheel_motor">
             <hardwareInterface>hardware_interface/EffortJointInterface</hardwareInterface>
-            <mechanicalReduction>1</mechanicalReduction>
-        </actuator>
-    </transmission>
-    <transmission name="tran2">
-        <type>transmission_interface/SimpleTransmission</type>
-        <joint name="joint1">
-            <hardwareInterface>hardware_interface/EffortJointInterface</hardwareInterface>
-        </joint>
-        <actuator name="left_front_wheel_motor">
-            <hardwareInterface>hardware_interface/EffortJointInterface</hardwareInterface>
-            <mechanicalReduction>-1</mechanicalReduction>
+            <mechanicalReduction>19.20</mechanicalReduction>
         </actuator>
     </transmission>
