Commit message: 新增框架工程moveit配置

File: sp_description/urdf/engineer_framed/engineer_chassis/engineer_chassis.xacro (robot description, xacro)
@@ -31,5 +31,5 @@
         izz="0.075914" />
     </inertial>
-    <!-- <visual>
+    <visual>
       <origin
         xyz="0 0 0"
@@ -44,6 +44,6 @@
           rgba="0.75294 0.75294 0.75294 1" />
       </material>
-    </visual> -->
-    <visual>
+    </visual>
+    <collision>
       <origin xyz="0 0 0.075" rpy="0 0 0" />
       <geometry>
@@ -55,13 +55,4 @@
           rgba="0.75294 0.75294 0.75294 1" />
       </material>
-    </visual>
-    <collision>
-      <origin
-        xyz="0 0 0"
-        rpy="0 0 0" />
-      <geometry>
-        <mesh
-          filename="package://sp_description/meshes/engineer_framed/engineer_chassis/base_link.STL" />
-      </geometry>
     </collision>
   </link>

File: sp_description/urdf/engineer_framed/engineer_manipulator_framed/engineer_manipulator_framed.xacro (robot description, xacro)
@@ -159,5 +159,5 @@
     <limit
       lower="0"
-      upper="0.86634"
+      upper="0.55"
       effort="20"
       velocity="5" />

Commit message: update PID for framed engineer

File: sp_description/urdf/engineer_framed/engineer_chassis/engineer_chassis.xacro (robot description, xacro)
@@ -46,7 +46,18 @@
     </visual>
     <collision>
-      <origin xyz="0 0 0.075" rpy="0 0 0" />
+      <origin xyz="0 0 0.090" rpy="0 0 0" />
       <geometry>
-        <box size="0.6 0.6 0.150"/>
+        <box size="0.6 0.6 0.120"/>
+      </geometry>
+      <material
+        name="">
+        <color
+          rgba="0.75294 0.75294 0.75294 1" />
+      </material>
+    </collision>
+    <collision>
+      <origin xyz="0 0 0.2" rpy="0 0 0" />
+      <geometry>
+        <box size="0.2 0.55 0.14"/>
       </geometry>
       <material

File: sp_description/urdf/engineer_framed/engineer_manipulator_framed/engineer_manipulator_framed.xacro (robot description, xacro)
@@ -38,11 +38,24 @@
     </visual>
     <collision>
-      <origin
-        xyz="0 0 0"
-        rpy="0 0 0" />
-      <geometry>
-        <mesh
-          filename="package://sp_description/meshes/engineer_framed/engineer_manipulator_framed/arm_base_link.STL" />
-      </geometry>
+      <origin xyz="0 0.27 0.25" rpy="0 0 0" />
+      <geometry>
+        <box size="0.40 0.04 0.42"/>
+      </geometry>
+      <material
+        name="">
+        <color
+          rgba="0.75294 0.75294 0.75294 1" />
+      </material>
+    </collision>
+    <collision>
+      <origin xyz="0 -0.27 0.25" rpy="0 0 0" />
+      <geometry>
+        <box size="0.4 0.04 0.42"/>
+      </geometry>
+      <material
+        name="">
+        <color
+          rgba="0.75294 0.75294 0.75294 1" />
+      </material>
     </collision>
   </link>
@@ -78,11 +91,68 @@
     </visual>
     <collision>
-      <origin
-        xyz="0 0 0"
-        rpy="0 0 0" />
-      <geometry>
-        <mesh
-          filename="package://sp_description/meshes/engineer_framed/engineer_manipulator_framed/link1.STL" />
-      </geometry>
+      <origin xyz="0 0.22 0.3" rpy="0 0 0" />
+      <geometry>
+        <box size="0.5 0.04 0.25"/>
+      </geometry>
+      <material
+        name="">
+        <color
+          rgba="0.75294 0.75294 0.75294 1" />
+      </material>
+    </collision>
+    <collision>
+      <origin xyz="0 -0.22 0.3" rpy="0 0 0" />
+      <geometry>
+        <box size="0.5 0.04 0.25"/>
+      </geometry>
+      <material
+        name="">
+        <color
+          rgba="0.75294 0.75294 0.75294 1" />
+      </material>
+    </collision>
+    <collision>
+      <origin xyz="0 0.18 0.4" rpy="0 0 0" />
+      <geometry>
+        <box size="0.7 0.06 0.06"/>
+      </geometry>
+      <material
+        name="">
+        <color
+          rgba="0.75294 0.75294 0.75294 1" />
+      </material>
+    </collision>
+    <collision>
+      <origin xyz="0 -0.18 0.4" rpy="0 0 0" />
+      <geometry>
+        <box size="0.7 0.06 0.06"/>
+      </geometry>
+      <material
+        name="">
+        <color
+          rgba="0.75294 0.75294 0.75294 1" />
+      </material>
+    </collision>
+    <collision>
+      <origin xyz="0.25 0 0.38" rpy="0 0 0" />
+      <geometry>
+        <box size="0.03 0.4 0.03"/>
+      </geometry>
+      <material
+        name="">
+        <color
+          rgba="0.75294 0.75294 0.75294 1" />
+      </material>
+    </collision>
+    <collision>
+      <origin xyz="-0.25 0 0.38" rpy="0 0 0" />
+      <geometry>
+        <box size="0.03 0.4 0.03"/>
+      </geometry>
+      <material
+        name="">
+        <color
+          rgba="0.75294 0.75294 0.75294 1" />
+      </material>
     </collision>
   </link>
@@ -333,7 +403,7 @@
     <limit
       lower="0"
-     upper="3.14"
-      effort="5"
-      velocity="5" />
+      upper="3.14"
+      effort="3"
+      velocity="15" />
   </joint>
   <link
@@ -392,6 +462,6 @@
      lower="-1.57"
       upper="1.57"
-      effort="5"
-      velocity="5" />
+      effort="3"
+      velocity="25" />
   </joint>
   <link
@@ -450,6 +520,6 @@
       lower="-3.14"
       upper="3.14"
-      effort="5"
-      velocity="5" />
+      effort="3"
+      velocity="25" />
   </joint>
    </xacro:macro>

File: sp_description/urdf/engineer_framed/manipulator_transmission.xacro (robot description, xacro)
@@ -13,8 +13,8 @@
         </transmission>
     </xacro:macro>
-   	<xacro:manipulator_transmission joint_name="joint1" mechanical_reduction="100"/>
-	<xacro:manipulator_transmission joint_name="joint2" mechanical_reduction="100"/>
-	<xacro:manipulator_transmission joint_name="joint3" mechanical_reduction="100"/>
-	<xacro:manipulator_transmission joint_name="joint4" mechanical_reduction="100"/>
+   	<xacro:manipulator_transmission joint_name="joint1" mechanical_reduction="723.71"/>
+	<xacro:manipulator_transmission joint_name="joint2" mechanical_reduction="1206.37"/>
+	<xacro:manipulator_transmission joint_name="joint3" mechanical_reduction="1206.37"/>
+	<xacro:manipulator_transmission joint_name="joint4" mechanical_reduction="400"/>
 	<xacro:manipulator_transmission joint_name="joint5" mechanical_reduction="1"/>
     <xacro:manipulator_transmission joint_name="joint6" mechanical_reduction="1"/>
