Commit message: Update moveit_servo to control the manipulator real-time by using topic 'delta_twist_cmd_' to control the pose and topic 'delta_joint_cmds' to control joints' angles.

File: sp_description/urdf/engineer_framed/engineer_manipulator_framed/engineer_manipulator_framed.xacro (robot description, xacro)
@@ -170,5 +170,5 @@
       xyz="0 0 1" />
     <limit
-      lower="-0.16"
+      lower="-0.15"
       upper="0"
       effort="150"
@@ -523,4 +523,18 @@
       velocity="25" />
   </joint>
+  <link name="vacuum_gripper"/>
+    <joint
+      name="vacuum_gripper_joint"
+      type="fixed">
+      <origin
+        xyz="0 0 0"
+        rpy="0 0 0" />
+      <parent
+        link="link7" />
+      <child
+        link="vacuum_gripper" />
+      <axis
+        xyz="0 0 1" />
+    </joint>
    </xacro:macro>
 </robot>
