Commit message: 新增syn_controller，用作控制电机同步运动

File: sp_description/urdf/engineer_manipulator/engineer.xacro (robot description, xacro)
@@ -1,18 +1,18 @@
 <?xml version="1.0"?>
 <robot xmlns:xacro="http://www.ros.org/wiki/xacro" name="engineer">
-    <xacro:include filename="$(find sp_description)/urdf/engineer_manipulator/engineer_manipulator/engineer_manipulator.xacro"/>
+    <!-- <xacro:include filename="$(find sp_description)/urdf/engineer_manipulator/engineer_manipulator/engineer_manipulator.xacro"/> -->
 	<xacro:include filename="$(find sp_description)/urdf/engineer_manipulator/engineer_chassis/engineer_chassis.xacro"/>
-	<xacro:include filename="$(find sp_description)/urdf/engineer_manipulator/manipulator_transmission.xacro"/>
+	<!-- <xacro:include filename="$(find sp_description)/urdf/engineer_manipulator/manipulator_transmission.xacro"/> -->
 	<xacro:include filename="$(find sp_description)/urdf/engineer_manipulator/fpv_module/fpv_module.xacro"/>
 	<xacro:arg name="use_simulation" default="true"/>
 	<xacro:engineer_chassis roller_type="simple"/>
 	<xacro:fpv_module/>
-	<xacro:engineer_manipulator/>
-<joint name="joint_arm2body" type="fixed">
+	<!-- <xacro:engineer_manipulator/>-->
+<!-- <joint name="joint_arm2body" type="fixed">
 		<axis xyz="0 0 1"/>
 		<origin xyz="0.022 0.166 0.228" rpy="0 0 -1.5708"/>
 		<parent link="base_link"/>
 		<child link="arm_base_link"/>
-	</joint>
+	</joint> -->
 	<joint name="joint_mast2body" type="fixed">
 			<axis xyz="0 0 1"/>

File: sp_description/urdf/engineer_manipulator/engineer_chassis/engineer_chassis.xacro (robot description, xacro)
@@ -111,8 +111,8 @@
                          wheel_z_offset="${wheel_offset_z}"
                          reflect="1" roller_type="${roller_type}"/>
-    <xacro:wheel_transmission prefix="left_front" mechanical_reduction="1"/>
+    <!-- <xacro:wheel_transmission prefix="left_front" mechanical_reduction="1"/>
     <xacro:wheel_transmission prefix="right_front" mechanical_reduction="-1"/>
     <xacro:wheel_transmission prefix="left_back" mechanical_reduction="1"/>
-    <xacro:wheel_transmission prefix="right_back" mechanical_reduction="-1"/>
+    <xacro:wheel_transmission prefix="right_back" mechanical_reduction="-1"/> -->
   </xacro:macro>
 `

File: sp_description/urdf/test/rmrobot.xacro (robot description, xacro)
@@ -35,9 +35,9 @@
         </inertial>
     </link>
-    <joint name="joint1" type="revolute">
+    <joint name="joint1" type="prismatic">
         <axis xyz="0 1 0"/>
         <origin xyz="0 ${width} ${height1 - axel_offset}" rpy="0 1.57 0"/>
              limit not work while type="continuous"
-        <limit effort="5." velocity="50." lower="-1e9" upper="1e9"/>
+        <limit effort="5." velocity="1.0" lower="-1e9" upper="1e9"/>
         <dynamics damping="0.01" friction="0.02"/>
         <parent link="link1"/>
@@ -66,4 +66,13 @@
         </inertial>
     </link>
+    <link name="test_link"/>
+    <joint name="joint2" type="revolute">
+        <axis xyz="0 1 0"/>
+        <origin xyz="0 0 0" rpy="0 1.57 0"/>
+        <limit effort="5." velocity="50." lower="-1e9" upper="1e9"/>
+        <dynamics damping="0.01" friction="0.02"/>
+        <parent link="link2"/>
+        <child link="test_link"/>
+    </joint>
     <transmission name="tran1">
         <type>transmission_interface/SimpleTransmission</type>
@@ -71,13 +80,46 @@
             <hardwareInterface>hardware_interface/EffortJointInterface</hardwareInterface>
         </joint>
-        <actuator name="right_front_wheel_motor">
+        <actuator name="motor1">
             <hardwareInterface>hardware_interface/EffortJointInterface</hardwareInterface>
             <mechanicalReduction>19.20</mechanicalReduction>
         </actuator>
     </transmission>
+     <transmission name="tran2">
+        <type>transmission_interface/SimpleTransmission</type>
+        <joint name="joint2">
+            <hardwareInterface>hardware_interface/EffortJointInterface</hardwareInterface>
+        </joint>
+        <actuator name="motor2">
+            <hardwareInterface>hardware_interface/EffortJointInterface</hardwareInterface>
+            <mechanicalReduction>-19.20</mechanicalReduction>
+        </actuator>
+    </transmission>
+    <!-- right_front_wheel_motor -->
+     <!-- <transmission name="differential_trans">
+        <type>transmission_interface/DifferentialTransmission</type>
+        <joint name="test_joint">
+            <role>joint1</role>
+            <hardwareInterface>hardware_interface/EffortJointInterface</hardwareInterface>
+        </joint>
+        <joint name="joint1">
+            <role>joint2</role>
+            <hardwareInterface>hardware_interface/EffortJointInterface</hardwareInterface>
+        </joint>
+        <actuator name="motor1">
+            <role>actuator1</role>
+            <mechanicalReduction>19.20</mechanicalReduction>
+        </actuator>
+        <actuator name="motor2">
+            <role>actuator2</role>
+            <mechanicalReduction>-19.20</mechanicalReduction>
+        </actuator>
+     </transmission> -->
     <gazebo>
         <plugin name="gazebo_ros_control" filename="libgazebo_ros_control.so">
             <robotNamespace>/</robotNamespace>
         </plugin>
+        <plugin name="adjustment_controller" filename="libadjustment_controller.so">
+			<robotNamespace>/</robotNamespace>
+		</plugin>
     </gazebo>
 </robot>
