Commit message: 更新manipulator_controller及其配套文件，实际效果待测
可使用遥控器单动各轴（应该重调PID）

File: sp_control/framed_moveit_config/config/gazebo_engineer_framed.urdf (robot description, URDF)
Before this commit: robot engineer_framed, 77 links, 76 joints
Links:
- added link fake_link1, mass 0.16243
- added link fake_link2, mass 3.3677
- added link fake_link3, mass 0.53167
- added link vacuum_gripper
- link arm_base_link: geometry collision box size=0.4 0.04 0.42; collision box size=0.40 0.04 0.42
- link base_link: geometry collision box size=0.2 0.55 0.14; collision box size=0.6 0.6 0.120
- link link1: geometry collision box size=0.03 0.4 0.03; collision box size=0.03 0.4 0.03
Joints:
- removed joint joint1
- removed joint joint2
- removed joint joint3
- added joint joint1_left: type prismatic, parent arm_base_link, child link1, origin xyz=0 0 0 rpy=0 0 0, axis 0 0 1, limit lower=-0.15 upper=0 effort=150 velocity=0.5
- added joint joint1_right: type prismatic, parent arm_base_link, child fake_link1, origin xyz=0 0 0 rpy=0 0 0, axis 0 0 1, limit lower=-0.15 upper=0 effort=150 velocity=0.5
- added joint joint2_left: type prismatic, parent link1, child link2, origin xyz=-0.7 0 0.3831 rpy=0 0 0, axis -1 0 0, limit lower=0 upper=0.55 effort=20 velocity=0.5
- added joint joint2_right: type prismatic, parent fake_link1, child fake_link2, origin xyz=-0.7 0 0.3831 rpy=0 0 0, axis -1 0 0, limit lower=0 upper=0.55 effort=20 velocity=0.5
- added joint joint3_left: type prismatic, parent link2, child link3, origin xyz=0.42794 0 0.072 rpy=0 3.3989E-05 0.01003, axis -1 0 0, limit lower=0 upper=0.4754 effort=20 velocity=0.5
- added joint joint3_right: type prismatic, parent fake_link2, child fake_link3, origin xyz=0.42794 0 0.072 rpy=0 3.3989E-05 0.01003, axis -1 0 0, limit lower=0 upper=0.4754 effort=20 velocity=0.5
- added joint vacuum_gripper_joint: type fixed, parent link7, child vacuum_gripper, origin xyz=0 0 0 rpy=0 0 0, axis 0 0 1
- joint joint4: limit lower=-0.3 upper=0.3 effort=0 velocity=0 -> lower=-0.3 upper=0.3 effort=20 velocity=0.5; origin xyz=0.50967 -0.005112 0.034017 rpy=0 -3.3987E-05 -0.01003 -> xyz=0.50967 -0.005112 0.034017 rpy=0 0 0
- joint joint5: limit lower=0 upper=3.14 effort=0 velocity=0 -> lower=0 upper=1.57 effort=3 velocity=3.14; origin xyz=0 -0.018 0.128 rpy=1.5708 0 0 -> xyz=0 -0.018 0.128 rpy=1.5708 -1.5708 0
- joint joint6: axis 0 0 -1 -> 0 0 1; limit lower=-1.57 upper=1.57 effort=0 velocity=0 -> lower=-1.57 upper=1.57 effort=3 velocity=3.14; origin xyz=0.07179 0 -0.028 rpy=1.5708 -1.5674 1.5708 -> xyz=0.07179 0 -0.028 rpy=1.5708 -1.5708 1.5708
- joint joint7: axis 0.033366 0 0.99944 -> 0 0 -1; limit lower=-3.14 upper=3.14 effort=20 velocity=5 -> lower=-3.14 upper=3.14 effort=3 velocity=3.14; origin xyz=0.00059574 -0.17579 -0.07179 rpy=1.5704 0 0.0033889 -> xyz=0 -0.17579 -0.07179 rpy=1.5708 3.1416 0

File: sp_description/urdf/engineer_framed/engineer_manipulator_framed/engineer_manipulator_framed.xacro (robot description, xacro)
@@ -158,5 +158,5 @@
   </link>
   <joint
-    name="joint1"
+    name="joint1_left"
     type="prismatic">
     <origin
@@ -173,5 +173,5 @@
       upper="0"
       effort="150"
-      velocity="5" />
+      velocity="0.5" />
   </joint>
   <link
@@ -216,5 +216,5 @@
   </link>
   <joint
-    name="joint2"
+    name="joint2_left"
     type="prismatic">
     <origin
@@ -231,5 +231,5 @@
       upper="0.55"
       effort="20"
-      velocity="5" />
+      velocity="0.5" />
   </joint>
   <link
@@ -274,5 +274,5 @@
   </link>
   <joint
-    name="joint3"
+    name="joint3_left"
     type="prismatic">
     <origin
@@ -289,5 +289,5 @@
       upper="0.4754"
       effort="20"
-      velocity="5" />
+      velocity="0.5" />
   </joint>
   <link
@@ -347,5 +347,5 @@
       upper="0.3"
       effort="20"
-      velocity="5" />
+      velocity="0.5" />
   </joint>
   <link
@@ -403,7 +403,7 @@
     <limit
       lower="0"
-      upper="3.14"
+      upper="1.57"
       effort="3"
-      velocity="15" />
+      velocity="3.14" />
   </joint>
   <link
@@ -463,5 +463,5 @@
       upper="1.57"
       effort="3"
-      velocity="25" />
+      velocity="3.14" />
   </joint>
   <link
@@ -521,5 +521,5 @@
       upper="3.14"
       effort="3"
-      velocity="25" />
+      velocity="3.14" />
   </joint>
   <link name="vacuum_gripper"/>
@@ -537,4 +537,106 @@
         xyz="0 0 1" />
     </joint>
+  <link name="fake_link1">
+    <inertial>
+        <origin
+          xyz="1.0099E-06 -0.062072 0.050902"
+          rpy="0 0 0" />
+        <mass
+          value="0.16243" />
+        <inertia
+          ixx="0.00010545"
+          ixy="-3.0539E-08"
+          ixz="1.4953E-08"
+          iyy="5.3443E-05"
+          iyz="-3.1729E-08"
+          izz="0.00014942" />
+      </inertial>
+    </link>
+  <joint
+    name="joint1_right"
+    type="prismatic">
+    <origin
+      xyz="0 0 0"
+      rpy="0 0 0" />
+    <parent
+      link="arm_base_link" />
+    <child
+      link="fake_link1" />
+    <axis
+      xyz="0 0 1" />
+    <limit
+      lower="-0.15"
+      upper="0"
+      effort="150"
+      velocity="0.5" />
+  </joint>
+  <link name="fake_link2">
+    <inertial>
+      <origin
+        xyz="0.73763 -0.012605 0.069937"
+        rpy="0 0 0" />
+      <mass
+        value="3.3677" />
+      <inertia
+        ixx="0.00060317"
+        ixy="-1.317E-07"
+        ixz="-5.0363E-06"
+        iyy="0.059389"
+        iyz="2.5076E-07"
+        izz="0.059509" />
+    </inertial>
+  </link>
+    <joint
+    name="joint2_right"
+    type="prismatic">
+    <origin
+      xyz="-0.7 0 0.3831"
+      rpy="0 0 0" />
+    <parent
+      link="fake_link1" />
+    <child
+      link="fake_link2" />
+    <axis
+      xyz="-1 0 0" />
+    <limit
+      lower="0"
+      upper="0.55"
+      effort="20"
+      velocity="0.5" />
+  </joint>
+  <link name="fake_link3">
+   <inertial>
+    <origin
+      xyz="0.51091 -0.0045583 0.038639"
+      rpy="0 0 0" />
+    <mass
+      value="0.53167" />
+    <inertia
+      ixx="0.0064927"
+      ixy="-6.4359E-05"
+      ixz="6.2407E-09"
+      iyy="0.00010061"
+      iyz="1.8149E-08"
+      izz="0.0065666" />
+    </inertial>
+  </link>
+  <joint
+    name="joint3_right"
+    type="prismatic">
+    <origin
+      xyz="0.42794 0 0.072"
+      rpy="0 3.3989E-05 0.01003" />
+    <parent
+      link="fake_link2" />
+    <child
+      link="fake_link3" />
+    <axis
+      xyz="-1 0 0" />
+    <limit
+      lower="0"
+      upper="0.4754"
+      effort="20"
+      velocity="0.5" />
+  </joint>
    </xacro:macro>
 </robot>

File: sp_description/urdf/engineer_framed/manipulator_transmission.xacro (robot description, xacro)
@@ -13,8 +13,11 @@
         </transmission>
     </xacro:macro>
-   	<xacro:manipulator_transmission joint_name="joint1" mechanical_reduction="723.71"/>
-	<xacro:manipulator_transmission joint_name="joint2" mechanical_reduction="1206.37"/>
-	<xacro:manipulator_transmission joint_name="joint3" mechanical_reduction="1206.37"/>
-	<xacro:manipulator_transmission joint_name="joint4" mechanical_reduction="768"/>
+   	<xacro:manipulator_transmission joint_name="joint1_left" mechanical_reduction="723.71"/>
+    <xacro:manipulator_transmission joint_name="joint1_right" mechanical_reduction="-723.71"/>
+	<xacro:manipulator_transmission joint_name="joint2_left" mechanical_reduction="603.18"/>
+    <xacro:manipulator_transmission joint_name="joint2_right" mechanical_reduction="-603.18"/>
+	<xacro:manipulator_transmission joint_name="joint3_left" mechanical_reduction="1206.37"/>
+    <xacro:manipulator_transmission joint_name="joint3_right" mechanical_reduction="-1206.37"/>
+	<xacro:manipulator_transmission joint_name="joint4" mechanical_reduction="400"/>
 	<xacro:manipulator_transmission joint_name="joint5" mechanical_reduction="1"/>
     <xacro:manipulator_transmission joint_name="joint6" mechanical_reduction="1"/>
