Commit message: 新增新工程模型与哨兵模型（需调整），并更新manipulator_controller以适应新工程

File: sp_description/urdf/engineer_framed/engineer.xacro (robot description, xacro)
@@ -1,15 +1,24 @@
 <?xml version="1.0"?>
 <robot xmlns:xacro="http://www.ros.org/wiki/xacro" name="engineer_framed">
-	<xacro:include filename="$(find sp_description)/urdf/engineer_framed/engineer_manipulator_framed/engineer_manipulator_framed.xacro"/>
+	<xacro:include filename="$(find sp_description)/urdf/engineer_framed/engineer_manipulator/engineer_manipulator.xacro"/>
 	<xacro:include filename="$(find sp_description)/urdf/engineer_framed/engineer_chassis/engineer_chassis.xacro"/>
+	<xacro:include filename="$(find sp_description)/urdf/engineer_framed/engineer_gimbal/engineer_gimbal.xacro"/>
 	<xacro:include filename="$(find sp_description)/urdf/engineer_framed/manipulator_transmission.xacro"/>
-    <xacro:engineer_manipulator_framed/>
     <xacro:engineer_chassis roller_type="simple"/>
-   	<joint name="joint_arm2body" type="fixed">
-		<axis xyz="0 0 1"/>
-		<origin xyz="-0.006 -0 0.12028" rpy="0 0 -1.57"/>
-		<parent link="base_link"/>
-		<child link="arm_base_link"/>
-	</joint>
+	<xacro:engineer_manipulator/>
+	<!-- <xacro:engineer_gimbal/> -->
+   	<joint name="z_base_joint" type="fixed">
+		<origin xyz="-5.6436E-05 0 0.13569" rpy="0 0 0" />
+		<parent link="base_link" />
+		<child link="z_base_link" />
+		<axis xyz="0 0 0" />
+  	</joint>
+	<!-- <joint name="gimbal_base_joint" type="fixed">
+		<origin
+		xyz="0.018 0.0825 0.029" rpy="0 0 0" />
+		<parent link="y_link" />
+		<child link="gimbal_base_link" />
+		<axis xyz="0 0 0" />
+  	</joint> -->
 	<!--在机器人模型的urdf/xacro文件中添加gazebo_ros_control插件-->
 	<gazebo>
@@ -20,4 +29,7 @@
 			<robotNamespace>/</robotNamespace>
 		</plugin>
+		<!-- <plugin name="gimbal_controller" filename="libgimbal_controller.so">
+			<robotNamespace>/</robotNamespace>
+		</plugin> -->
 	</gazebo>
 </robot>

File: sp_description/urdf/engineer_framed/engineer_chassis/engineer_chassis.xacro (robot description, xacro)
@@ -7,27 +7,27 @@
   xmlns:xacro="http://wiki.ros.org/xacro">
   <xacro:include filename="$(find sp_description)/urdf/common/mecanum_wheel.xacro"/>
-  <xacro:property name="wheel_front" value="0.19185"/>
-  <xacro:property name="wheel_back" value="-0.19152"/>
-  <xacro:property name="wheel_left" value="0.221"/>
-  <xacro:property name="wheel_right" value="-0.221"/>
+  <xacro:property name="wheel_front" value="0.19463"/>
+  <xacro:property name="wheel_back" value="-0.19463"/>
+  <xacro:property name="wheel_left" value="0.227 "/>
+  <xacro:property name="wheel_right" value="-0.227 "/>
   <xacro:property name="wheel_offset_z" value="0.077"/>
   <xacro:property name="wheel_joint_damping" value="1.0"/>
   <xacro:property name="wheel_joint_friction" value="1.0"/>
   <xacro:macro name="engineer_chassis" params="roller_type">
-   <link
+  <link
     name="base_link">
     <inertial>
       <origin
-        xyz="0.047614 -0.013852 0.13893"
+        xyz="0.0234504860983126 0.00205520120472003 0.106854712514192"
         rpy="0 0 0" />
       <mass
-        value="12.232" />
+        value="10.2607853738169" />
       <inertia
-        ixx="0.039383"
-        ixy="2.7131E-05"
-        ixz="0.00010315"
-        iyy="0.048017"
-        iyz="0.00051335"
-        izz="0.075914" />
+        ixx="0.0251253323940971"
+        ixy="0.00026008044804615"
+        ixz="2.48842772985471E-05"
+        iyy="0.0390351483919132"
+        iyz="-6.80934351257943E-05"
+        izz="0.0558214144240648" />
     </inertial>
     <visual>
@@ -42,28 +42,15 @@
         name="">
         <color
-          rgba="0.75294 0.75294 0.75294 1" />
+          rgba="0.792156862745098 0.819607843137255 0.933333333333333 1" />
       </material>
     </visual>
     <collision>
-      <origin xyz="0 0 0.090" rpy="0 0 0" />
+      <origin
+        xyz="0 0 0"
+        rpy="0 0 0" />
       <geometry>
-        <box size="0.6 0.6 0.120"/>
+        <mesh
+          filename="package://sp_description/meshes/engineer_framed/engineer_chassis/base_link.STL" />
       </geometry>
-      <material
-        name="">
-        <color
-          rgba="0.75294 0.75294 0.75294 1" />
-      </material>
-    </collision>
-    <collision>
-      <origin xyz="0 0 0.2" rpy="0 0 0" />
-      <geometry>
-        <box size="0.2 0.55 0.14"/>
-      </geometry>
-      <material
-        name="">
-        <color
-          rgba="0.75294 0.75294 0.75294 1" />
-      </material>
     </collision>
   </link>
@@ -84,8 +71,8 @@
                          wheel_z_offset="${wheel_offset_z}"
                          reflect="1" roller_type="${roller_type}"/>
-    <!-- <xacro:wheel_transmission prefix="left_front" mechanical_reduction="19.2032"/>
+    <xacro:wheel_transmission prefix="left_front" mechanical_reduction="19.2032"/>
     <xacro:wheel_transmission prefix="right_front" mechanical_reduction="-19.2032"/>
     <xacro:wheel_transmission prefix="left_back" mechanical_reduction="19.2032"/>
-    <xacro:wheel_transmission prefix="right_back" mechanical_reduction="-19.2032"/> -->
+    <xacro:wheel_transmission prefix="right_back" mechanical_reduction="-19.2032"/>
   </xacro:macro>
 </robot>

File: sp_description/urdf/engineer_framed/manipulator_transmission.xacro (robot description, xacro)
@@ -13,13 +13,12 @@
         </transmission>
     </xacro:macro>
-   	<xacro:manipulator_transmission joint_name="joint1_left" mechanical_reduction="723.71"/>
-    <xacro:manipulator_transmission joint_name="joint1_right" mechanical_reduction="-723.71"/>
-	<xacro:manipulator_transmission joint_name="joint2_left" mechanical_reduction="603.18"/>
-    <xacro:manipulator_transmission joint_name="joint2_right" mechanical_reduction="-603.18"/>
-	<xacro:manipulator_transmission joint_name="joint3_left" mechanical_reduction="1206.37"/>
-    <xacro:manipulator_transmission joint_name="joint3_right" mechanical_reduction="-1206.37"/>
-	<xacro:manipulator_transmission joint_name="joint4" mechanical_reduction="400"/>
-	<xacro:manipulator_transmission joint_name="joint5" mechanical_reduction="1"/>
-    <xacro:manipulator_transmission joint_name="joint6" mechanical_reduction="1"/>
-    <xacro:manipulator_transmission joint_name="joint7" mechanical_reduction="1"/>
+   	<xacro:manipulator_transmission joint_name="z_joint_left" mechanical_reduction="1"/>
+    <xacro:manipulator_transmission joint_name="z_joint_right" mechanical_reduction="-1"/>
+	<xacro:manipulator_transmission joint_name="x_joint_left" mechanical_reduction="1"/>
+    <xacro:manipulator_transmission joint_name="x_joint_right" mechanical_reduction="-1"/>
+	<xacro:manipulator_transmission joint_name="y_joint" mechanical_reduction="1"/>
+	<xacro:manipulator_transmission joint_name="yaw_joint" mechanical_reduction="1"/>
+	<xacro:manipulator_transmission joint_name="roll1_joint" mechanical_reduction="1"/>
+    <xacro:manipulator_transmission joint_name="pitch_joint" mechanical_reduction="1"/>
+    <xacro:manipulator_transmission joint_name="roll2_joint" mechanical_reduction="-1"/>
 </robot>

File: sp_description/urdf/test/rmrobot.xacro (robot description, xacro)
@@ -35,5 +35,5 @@
         </inertial>
     </link>
-    <joint name="joint1" type="prismatic">
+    <joint name="joint1" type="revolute">
         <axis xyz="0 1 0"/>
         <origin xyz="0 ${width} ${height1 - axel_offset}" rpy="0 1.57 0"/>
@@ -82,5 +82,5 @@
         <actuator name="motor1">
             <hardwareInterface>hardware_interface/EffortJointInterface</hardwareInterface>
-            <mechanicalReduction>19.20</mechanicalReduction>
+            <mechanicalReduction>1</mechanicalReduction>
         </actuator>
     </transmission>
@@ -92,5 +92,5 @@
         <actuator name="motor2">
             <hardwareInterface>hardware_interface/EffortJointInterface</hardwareInterface>
-            <mechanicalReduction>-19.20</mechanicalReduction>
+            <mechanicalReduction>-1</mechanicalReduction>
         </actuator>
     </transmission>

Commit message: 更新MANL模式
（1）读取IMU空间角速度解算为小臂各轴速度
（2）暂时屏蔽AUTO模式
（3）底层中断逻辑修改（待测）
（4）整理rotate_ore_controlller

File: sp_description/urdf/engineer_framed/engineer.xacro (robot description, xacro)
@@ -8,4 +8,5 @@
     <xacro:engineer_chassis roller_type="simple"/>
 	<xacro:engineer_manipulator/>
+	<xacro:engineer_rotating_ore/>
 	<!-- <xacro:engineer_gimbal/> -->
    	<joint name="z_base_joint" type="fixed">

File: sp_description/urdf/engineer_framed/engineer_manipulator/engineer_manipulator.xacro (robot description, xacro)
@@ -390,6 +390,6 @@
       xyz="0 1 0" />
     <limit
-      lower="-1e9"
-      upper="1e9"
+      lower="-3.14"
+      upper="3.14"
       effort="2"
       velocity="5" />
@@ -446,8 +446,8 @@
       link="roll2_link" />
     <axis
-      xyz="-1 0 0" />
-    <limit
-      lower="-1e9"
-      upper="1e9"
+      xyz="1 0 0" />
+    <limit
+      lower="-6.28"
+      upper="6.28"
       effort="2"
       velocity="5" />

File: sp_description/urdf/engineer_framed/engineer_rotating_ore/engineer_rotating_ore.xacro (robot description, xacro)
@@ -7,78 +7,52 @@
   xmlns:xacro="http://wiki.ros.org/xacro">
   <xacro:macro name="engineer_rotating_ore">
-  <link
-    name="ore_link">
-    <inertial>
-      <origin
-        xyz="-0.0502503997952509 0.00270734420696059 0.158256772820509"
-        rpy="0 0 0" />
-      <mass
-        value="6.17465462282344" />
-      <inertia
-        ixx="0.0492802144410084"
-        ixy="1.5051986903972E-07"
-        ixz="0.000188405207234761"
-        iyy="0.060278709466721"
-        iyz="-8.44201370846196E-06"
-        izz="0.0135632849138947" />
-    </inertial>
-    <visual>
-      <origin
-        xyz="0 0 0"
-        rpy="0 0 0" />
-      <geometry>
-        <mesh
-          filename="package://sp_description/meshes/engineer_framed/engineer_manipulator/z_link.STL" />
-      </geometry>
-      <material
-        name="">
-        <color
-          rgba="0.752941176470588 0.752941176470588 0.752941176470588 1" />
-      </material>
-    </visual>
-    <collision>
-      <origin
-        xyz="0 0 0"
-        rpy="0 0 0" />
-      <geometry>
-        <mesh
-          filename="package://sp_description/meshes/engineer_framed/engineer_manipulator/z_link.STL" />
-      </geometry>
-    </collision>
-  </link>
-  <joint
-    name="ore_left"
-    type="revolute">
-    <origin
-      xyz="0 0 0"
-      rpy="0 0 0" />
-    <child
-      link="ore_link" />
-    <axis
-      xyz="0 0 1" />
-    <limit
-      lower="0"
-      upper="11"
-      effort="10"
-      velocity="1" />
-  </joint>
-    <joint
-    name="ore_right"
-    type="revolute">
-    <origin
-      xyz="0 0 0"
-      rpy="0 0 0" />
-    <parent
-      link="z_base_link" />
-    <child
-      link="fake_z_link" />
-    <axis
-      xyz="0 0 1" />
-    <limit
-      lower="0"
-      upper="11"
-      effort="10"
-      velocity="1" />
-  </joint>
-</xacro:macro>
+    <link name="ore_left_link">
+      <inertial>
+        <origin xyz="0 0 0" rpy="0 0 0"/>
+        <mass value="0.013"/>
+        <inertia ixx="0.001" ixy="0.0" ixz="0.0" iyy="0.001" iyz="0.0" izz="0.001"/>
+      </inertial>
+    </link>
+    <link name="ore_right_link">
+      <inertial>
+        <origin xyz="0 0 0" rpy="0 0 0"/>
+        <mass value="0.013"/>
+        <inertia ixx="0.001" ixy="0.0" ixz="0.0" iyy="0.001" iyz="0.0" izz="0.001"/>
+      </inertial>
+    </link>
+    <joint name="ore_left_joint" type="revolute">
+      <origin xyz="0 0 0" rpy="0 0 0" />
+      <parent link="z_base_link" />
+      <child link="ore_left_link" />
+      <axis xyz="0 0 1" />
+      <limit lower="0" upper="11" effort="10" velocity="1" />
+    </joint>
+    <joint name="ore_right_joint" type="revolute">
+      <origin xyz="0 0 0" rpy="0 0 0" />
+      <parent link="z_base_link" />
+      <child link="ore_right_link" />
+      <axis xyz="0 0 1" />
+      <limit lower="0" upper="11" effort="10" velocity="1" />
+    </joint>
+    <transmission name="trans_ore_left_joint" >
+      <type>transmission_interface/SimpleTransmission</type>
+      <actuator name="ore_left_joint_motor">
+        <mechanicalReduction>-1</mechanicalReduction>
+        <hardwareInterface>hardware_interface/EffortJointInterface</hardwareInterface>
+      </actuator>
+			<joint name="ore_left_joint">
+				<hardwareInterface>hardware_interface/EffortJointInterface</hardwareInterface>
+			</joint>
+    </transmission>
+    <transmission name="trans_ore_right_joint" >
+      <type>transmission_interface/SimpleTransmission</type>
+      <actuator name="ore_right_joint_motor">
+        <mechanicalReduction>1</mechanicalReduction>
+        <hardwareInterface>hardware_interface/EffortJointInterface</hardwareInterface>
+      </actuator>
+			<joint name="ore_right_joint">
+				<hardwareInterface>hardware_interface/EffortJointInterface</hardwareInterface>
+			</joint>
+    </transmission>
+  </xacro:macro>
 </robot>

File: sp_description/urdf/engineer_framed/manipulator_transmission.xacro (robot description, xacro)
@@ -18,9 +18,7 @@
     <xacro:manipulator_transmission joint_name="x_joint_right" mechanical_reduction="-2010.62"/>
 	<xacro:manipulator_transmission joint_name="y_joint" mechanical_reduction="274.285"/>
-<xacro:manipulator_transmission joint_name="yaw_joint" mechanical_reduction="1"/>
+    <xacro:manipulator_transmission joint_name="yaw_joint" mechanical_reduction="1"/>
 	<xacro:manipulator_transmission joint_name="roll1_joint" mechanical_reduction="1"/>
     <xacro:manipulator_transmission joint_name="pitch_joint" mechanical_reduction="1.5"/>
     <xacro:manipulator_transmission joint_name="roll2_joint" mechanical_reduction="-1.5"/>
-   	<xacro:manipulator_transmission joint_name="ore_left" mechanical_reduction="-1"/>
-   	<xacro:manipulator_transmission joint_name="ore_right" mechanical_reduction="1"/>
 </robot>

File: sp_description/urdf/engineer_manipulator/engineer_chassis/engineer_chassis.xacro (robot description, xacro)
@@ -111,8 +111,8 @@
                          wheel_z_offset="${wheel_offset_z}"
                          reflect="1" roller_type="${roller_type}"/>
-    <!-- <xacro:wheel_transmission prefix="left_front" mechanical_reduction="1"/>
-    <xacro:wheel_transmission prefix="right_front" mechanical_reduction="-1"/>
-    <xacro:wheel_transmission prefix="left_back" mechanical_reduction="1"/>
-    <xacro:wheel_transmission prefix="right_back" mechanical_reduction="-1"/> -->
+    <!-- <xacro:wheel_transmission prefix="left_front" mechanical_reduction="19.20"/>
+    <xacro:wheel_transmission prefix="right_front" mechanical_reduction="-19.20"/>
+    <xacro:wheel_transmission prefix="left_back" mechanical_reduction="19.20"/>
+    <xacro:wheel_transmission prefix="right_back" mechanical_reduction="-19.20"/> -->
   </xacro:macro>
 `

Commit message: Update syn_controller and adjust PID for z axis, fix z axis shaking problem

File: sp_description/urdf/engineer_framed/engineer.xacro (robot description, xacro)
@@ -9,5 +9,5 @@
 	<xacro:engineer_manipulator/>
 	<xacro:engineer_rotating_ore/>
-	<!-- <xacro:engineer_gimbal/> -->
+	<xacro:engineer_gimbal/>
    	<joint name="z_base_joint" type="fixed">
 		<origin xyz="-5.6436E-05 0 0.13569" rpy="0 0 0" />
@@ -16,5 +16,5 @@
 		<axis xyz="0 0 0" />
   	</joint>
-	<!-- <joint name="gimbal_base_joint" type="fixed">
+	<joint name="gimbal_base_joint" type="fixed">
 		<origin
 		xyz="0.018 0.0825 0.029" rpy="0 0 0" />
@@ -22,5 +22,5 @@
 		<child link="gimbal_base_link" />
 		<axis xyz="0 0 0" />
-  	</joint> -->
+  	</joint>
 	<!--在机器人模型的urdf/xacro文件中添加gazebo_ros_control插件-->
 	<gazebo>
@@ -31,7 +31,7 @@
 			<robotNamespace>/</robotNamespace>
 		</plugin>
-		<!-- <plugin name="gimbal_controller" filename="libgimbal_controller.so">
+		<plugin name="gimbal_controller" filename="libgimbal_controller.so">
 			<robotNamespace>/</robotNamespace>
-		</plugin> -->
+		</plugin>
 	</gazebo>
 </robot>
